File: cd_rom_mech.kicad_sch (KiCad schematic)
At the start: 11 parts, among them IC1 BA6290A, IC101 CXA1081, IC102 CXA1082BQ, IC107 RC4558, IC2 BA6290A, IC201 LC7881M, IC202 RC4558, IC203 RC4558, P1 Conn_01x08, P2 Conn_01x08

Commit message: More tracing.
Parts:
- added R105: ?, Resistor_SMD:R_0805_2012Metric, symbol Device:R
Connections:
- net TE: now reaches IC102.45 (TE)
- net TZC: now reaches IC102.46 (TZC)
- net ATSC: now reaches IC102.47 (ATSC)
Changed lines of the file:
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@@
+    (stroke (width 0) (type default))
+  )
+  (wire (pts (xy 47.625 199.39) (xy 54.61 199.39))
+    (stroke (width 0) (type default))
+  )
+  (wire (pts (xy 40.005 201.93) (xy 54.61 201.93))
     (stroke (width 0) (type default))
   )
@@
     (stroke (width 0) (type default))
   )
+  (wire (pts (xy 40.005 196.85) (xy 54.61 196.85))
+    (stroke (width 0) (type default))
+  )
   (wire (pts (xy 365.76 62.23) (xy 370.84 62.23))
     (stroke (width 0) (type default))
@@
   (wire (pts (xy 128.27 184.15) (xy 143.51 184.15))
     (stroke (width 0) (type default))
+  )
+  (global_label "TZC" (shape input) (at 47.625 199.39 180) (fields_autoplaced)
+    (effects (font (size 1.27 1.27)) (justify right))
+    (property "Intersheetrefs" "${INTERSHEET_REFS}" (at 41.1927 199.39 0)
+      (effects (font (size 1.27 1.27)) (justify right) hide)
+    )
+  )
+  (global_label "TE" (shape input) (at 40.005 196.85 180) (fields_autoplaced)
+    (effects (font (size 1.27 1.27)) (justify right))
+    (property "Intersheetrefs" "${INTERSHEET_REFS}" (at 34.9032 196.85 0)
+      (effects (font (size 1.27 1.27)) (justify right) hide)
+    )
+  )
+  (global_label "ATSC" (shape input) (at 40.005 201.93 180) (fields_autoplaced)
+    (effects (font (size 1.27 1.27)) (justify right))
+    (property "Intersheetrefs" "${INTERSHEET_REFS}" (at 32.4841 201.93 0)
+      (effects (font (size 1.27 1.27)) (justify right) hide)
+    )
   )
   (symbol (lib_id "Amplifier_Operational:RC4558") (at 182.88 149.86 0) (unit 1)
@@
         )
       )
+    )
+  )
+  (symbol (lib_id "Device:R") (at 141.605 132.08 270) (unit 1)
+    (in_bom yes) (on_board yes) (dnp no) (fields_autoplaced)
+    (property "Reference" "R105" (at 141.605 127 90)
+      (effects (font (size 1.27 1.27)))
+    )
+    (property "Value" "?" (at 141.605 129.54 90)
+      (effects (font (size 1.27 1.27)))
+    )
+    (property "Footprint" "Resistor_SMD:R_0805_2012Metric" (at 141.605 130.302 90)
+      (effects (font (size 1.27 1.27)) hide)
+    )
+    (property "Datasheet" "~" (at 141.605 132.08 0)
+      (effects (font (size 1.27 1.27)) hide)
+    )
+    (pin "1")
+    (pin "2")
+    (instances
+      (project "PCE"
+        (path "/c1c718c6-a427-431e-a18b-e46f94ae8e09/1d91d06a-381a-4a70-bfc1-2abf4d159a91"
+          (reference "R105") (unit 1)
+        )
+        (path "/c1c718c6-a427-431e-a18b-e46f94ae8e09/bb2f9872-1813-43e0-bcfc-5c5426bf43ce"
+          (reference "R121") (unit 1)
+        )
+      )

Commit message: Yet more tracing.
Parts:
- added C105 (x2): ~, A-PCENGINE:Elec_P5.00mm, symbol Device:C_Polarized
- added P3: Conn_01x07, Connector_PinHeader_2.00mm:PinHeader_1x07_P2.00mm_Vertical, symbol Connector_Generic:Conn_01x07
Connections:
- net GND is gone; now on net GNDA: IC1.12 (GND), IC2.12 (GND)
- net +9V: now also C105.1
- net GNDA: now reaches IC107.2 (-)
- net GNDA: now also IC107.3 (+), IC107.4 (V-), IC201.12 (TST1), IC201.13 (TST2), IC201.15 (GND), IC201.17 (GND), IC201.18 (VREFL2), IC201.5 (WCLK2), C105.2, C105.2, P3.5 (Pin_5)
- net at IC107.5 (+): now also IC2.6 (E+)
- net at IC107.8 (V+): now also C105.1
- net at IC201.3 (VREFH2): now also IC201.4 (VDD)
- net at IC102.11 (TAO): now also IC102.13 (SL+)
- net TA-: now reaches IC102.12 (TA-)
- net FGD: now reaches IC102.2 (FGD)
- net at IC102.28 (PDI): now also IC102.31 (3.5V)
- net FS3: now reaches IC102.3 (FS3)
- net FLB: now reaches IC102.4 (FLB)
- net FE0: now reaches IC102.5 (FEO)
- net FE-: now reaches IC102.6 (FE-)
- net SRCH: now reaches IC102.7 (SRCH)
- net TGU: now reaches IC102.8 (TGU)
- net TG2: now reaches IC102.9 (TG2)
Other:
- moved on the sheet: IC107A, IC107B

Commit message: Power rails, etc.
Parts:
- added C105: ?, Capacitor_SMD:C_0805_2012Metric, symbol Device:C
- added R105 (x2): ?, Resistor_SMD:R_0805_2012Metric, symbol Device:R
Connections:
- net +9V: now also C105.1
- net GNDA: now also P2.1 (Pin_1)
- net at IC107.5 (+), IC2.6 (E+): now also IC1.6 (E+)
- net at IC107.8 (V+): no longer C105.1
- net at IC1.10 (OUTA1): now also P2.6 (Pin_6)
- net at IC1.11 (OUT1): now also IC1.9 (INA1), P2.5 (Pin_5)
- net at IC1.2 (OUT0), IC1.4 (INA0): now also P2.7 (Pin_7)
- net at IC1.3 (OUTA0): now also P2.8 (Pin_8)
- net XRST: now reaches R105.1
- net XRST: now also R105.2
- net at R105.2: now also R105.2
- net at P3.1 (Pin_1): now also IC2.10 (OUTA1)
- net at P3.2 (Pin_2): now also IC2.11 (OUT1), IC2.9 (INA1)
- net at P3.6 (Pin_6): now also IC2.3 (OUTA0)
- net at P3.7 (Pin_7): now also IC2.2 (OUT0), IC2.4 (INA0)
- net SENS: now reaches IC102.30 (VCOF)
- net CNIN: now reaches IC102.32 (C864)
- net at IC102.34 (MDP): now also C105.1, R105.1
- net DATA: now reaches IC102.35 (MON)
- net FSW: now reaches IC102.36 (FSW)
- net FSW: now also R105.1
- net DVCC: now reaches IC102.37 (DVCC)
Other:
- moved on the sheet: C105, IC107B, P2, R105

Commit message: IC routing mostly complete, start adding passives.
Parts:
- added C105 (x6): ?, A-PCENGINE:SMD_0805_Narrow, symbol Device:C
- added C105: ?, A-PCENGINE:SMD_0805_Narrow_Long, symbol Device:C
- added P5: Conn_01x05, Connector_PinHeader_2.00mm:PinHeader_1x06_P2.00mm_Vertical, symbol Connector_Generic:Conn_01x06
- added R105 (x5): ?, A-PCENGINE:SMD_0805_Narrow, symbol Device:R
- C105: footprint Capacitor_SMD:C_0805_2012Metric -> A-PCENGINE:SMD_0805_Narrow
- IC101: footprint Package_SO:SSOP-32_11.305x20.495mm_P1.27mm -> A-PCENGINE:SSOP-30_P1.27mm
- R105: footprint Resistor_SMD:R_0805_2012Metric -> A-PCENGINE:SMD_0805_Narrow
Connections:
- net FLB is gone; now on net WCLK: IC102.4 (FLB)
- net DATA: now also IC102.23 (DATA), R105.1, C105.1, R105.1; no longer IC102.35 (MON)
- net FE-: now also IC101.22 (MIRR)
- net FE0: now also IC101.28 (FOK)
- net GNDA: now also IC202.4 (V-), IC203.4 (V-)
- net TGU: now also IC101.21 (DEFECT)
- net at IC202.6 (-): now also IC202.7
- net at IC102.24 (XLT): now also R105.2, C105.2, R105.1; no longer R105.1
- net at IC101.10 (F): now also P1.7 (Pin_7)
- net at IC101.11 (E): now also P1.8 (Pin_8)
- net at IC101.14 (VR): now also IC101.9 (VC)
- net GND: now reaches IC101.17 (VEE)
- net at IC101.2 (RFO): now also P5.2 (Pin_2)
- net at IC101.20 (TE): now also P5.3 (Pin_3)
- net at IC101.25 (DGND): now also P5.6 (Pin_6)
- net EFM: now reaches IC101.27 (EFM)
- net at IC101.29 (~{LD_ON}): now also P5.4 (Pin_4)
- net +5VD: now reaches IC101.30 (VCC)
- net PD: now reaches IC101.6 (PD)
- net PD: now also P2.3 (Pin_3)
- net at IC101.7 (PD1): now also P1.4 (Pin_4)
- net at IC101.8 (PD2): now also P1.3 (Pin_3)
- net P3P4: now reaches P3.4 (Pin_4)
- net +5VP: now reaches IC203.8 (V+)
- net +5VP: now also IC202.8 (V+)
- net at IC202.1: now also IC202.2 (-)
- net LRCK: now reaches IC201.6 (LRCK)
- net WCLK: now reaches IC201.7 (WCLK1)
- net BCLK: now reaches IC201.9 (BCLK)
- net at IC102.10 (AVCC): now also C105.1
- net SL+: now reaches IC102.11 (TAO), IC102.13 (SL+)
- net SL+: now also C105.1, P5.1 (Pin_1)
- net at IC102.14 (SLO): now also C105.2
- net at IC102.15 (SL-): now also C105.1
- net at IC102.16 (SSTOP): now also C105.2
- net at IC102.17 (FSET): now also C105.1, R105.1
- net at IC102.18 (SENS): now also C105.2, R105.2, R105.2
- net at IC102.20 (C.OUT): now also C105.1
- net at IC102.21 (DIRC): now also C105.2
- net at IC102.25 (CLK): now also C105.2, R105.2
- new net: P5.5 (Pin_5), R105.1
- new net ASY: R105.2
- new net MON: IC102.35 (MON)
- new net P7P5: R105.1
- new net P7P6: R105.2
Other:
- moved on the sheet: C105, IC101, IC107A, IC107C, IC202C, P1, R105

Commit message: Bunch of passives and what-not.
Parts:
- added C105 (x4), C138 (x6): ?, A-PCENGINE:SMD_0805_Narrow_Long, symbol Device:C
- added C127: C, A-PCENGINE:SMD_1806, symbol Device:C
- added C138: ?, A-PCENGINE:SMD_1206, symbol Device:C
- added R105 (x28): ?, A-PCENGINE:SMD_0805_Narrow_Long, symbol Device:R
- added R105 (x2): ?, A-PCENGINE:SMD_0805_Narrow, symbol Device:R
- added TP1, TP10, TP11, TP12, TP2, TP3, TP4, TP5, TP6, TP7: ~, A-PCENGINE:Test_Point_1.5mm, symbol Connector:TestPoint
- C105, R105: footprint A-PCENGINE:SMD_0805_Narrow -> A-PCENGINE:SMD_0805_Narrow_Long
Connections:
- net FGD is gone; now on an unnamed net: IC102.2 (FGD)
- net FS3 is gone; now on an unnamed net: IC102.3 (FS3)
- net SRCH is gone; now on net GND: IC102.7 (SRCH)
- net TA- is gone; now on an unnamed net: IC102.12 (TA-)
- net TG2 is gone; now on an unnamed net: IC102.9 (TG2)
- net TZC is gone; now on an unnamed net: IC102.46 (TZC)
- net +5VD: now also IC102.37 (DVCC), C138.2
- net +9V: now also R105.1
- net ATSC: now also C105.1, C105.1, IC102.1 (VC), P1.5 (Pin_5), P5.1 (Pin_1), R105.1, R105.2
- net CNIN: now also IC102.20 (C.OUT); no longer IC102.32 (C864)
- net DATA: no longer C105.1, R105.1, R105.1
- net DVCC: now also IC102.25 (CLK); no longer IC102.37 (DVCC)
- net FSW: now also C138.2, R105.1; no longer IC102.36 (FSW), R105.1
- net GND: now also IC102.16 (SSTOP), IC102.19 (AVEE), IC102.26 (DGND), C138.1, C138.1, C138.1, C138.2, R105.2
- net GNDA: now also R105.2, TP5.1
- net P3P4: now also TP4.1
- net SENS: now also IC102.18 (SENS); no longer IC102.30 (VCOF)
- net WCLK: now also IC102.40 (WDCK); no longer IC102.4 (FLB)
- net at C105.2, R105.2: now also IC102.13 (SL+); no longer IC102.25 (CLK)
- net at C105.2, R105.1, R105.2: no longer IC102.24 (XLT)
- net at IC1.6 (E+), IC107.5 (+), IC2.6 (E+): now also R105.1, R105.2
- net at IC107.6 (-): now also R105.2, R105.2
- net at IC107.7: now also R105.1, R105.1, R105.1, R105.1, R105.2, TP12.1
- net at R105.2: no longer R105.2
- net at C105.1: now also IC102.8 (TGU); no longer IC102.20 (C.OUT)
- net at C105.2: no longer IC102.21 (DIRC)
- net at IC1.11 (OUT1), IC1.9 (INA1), P2.5 (Pin_5): now also C105.2, R105.2
- net at IC1.2 (OUT0), IC1.4 (INA0), P2.7 (Pin_7): now also C105.1, R105.2
- net at IC1.5 (IN0): now also R105.1, R105.1, R105.2, R105.2
- net at IC1.8 (IN1): now also R105.1, R105.1, R105.1, R105.2
- net at C105.2: now also IC102.4 (FLB); no longer IC102.16 (SSTOP)
- net at IC101.2 (RFO), P5.2 (Pin_2): now also TP10.1
- net at IC101.29 (~{LD_ON}), P5.4 (Pin_4): now also TP11.1
- net at C105.1: no longer IC102.15 (SL-)
- net at C105.2: no longer IC102.14 (SLO)
- net at IC101.19 (FE): now also R105.1
- net at IC101.7 (PD1), P1.4 (Pin_4): now also P1.1 (Pin_1)
- net at IC101.8 (PD2), P1.3 (Pin_3): now also P1.2 (Pin_2)
- net at C105.1: no longer IC102.10 (AVCC)
- net at IC2.10 (OUTA1), P3.1 (Pin_1): now also C105.1, TP1.1
- net at IC2.11 (OUT1), IC2.9 (INA1), P3.2 (Pin_2): now also C105.2, R105.2, TP2.1
- net P3P3: now reaches P3.3 (Pin_3)
- net P3P3: now also TP3.1
- net at IC2.3 (OUTA0), P3.6 (Pin_6): now also C105.1, TP6.1
- net at IC2.2 (OUT0), IC2.4 (INA0), P3.7 (Pin_7): now also C105.2, R105.2, TP7.1
- net at IC2.5 (IN0): now also R105.1, R105.1, R105.1
- net at IC2.8 (IN1): now also R105.1, R105.1, R105.2
- net at C105.2, R105.2, R105.2: now also IC102.6 (FE-); no longer IC102.18 (SENS)
- net FEO: now reaches C105.1, R105.1
- net FEO: now also IC102.5 (FEO), R105.2; no longer IC102.17 (FSET)
- net at IC102.22 (XRST): now also C105.1, R105.1
- net at IC102.27 (BW): now also C127.1, C138.2
- net at IC102.31 (3.5V): now also R105.1; no longer IC102.28 (PDI)
- net at IC102.29 (ISET): now also R105.2
- net LOCK: now reaches IC102.33 (LOCK)
- net at IC102.38 (SPDL-): now also R105.2
- net SDPLO: now reaches IC102.39 (SPDLO)
- net SDPLO: now also R105.1, R105.2
- net FOK: now reaches IC102.41 (FOK)
- net FOK: now also IC101.28 (FOK)
- net MIRR: now reaches IC102.42 (MIRR)
- net MIRR: now also IC101.22 (MIRR)
- net DFCT: now reaches IC102.44 (DFCT)
- net DFCT: now also IC101.21 (DEFECT)
- net FE: now reaches IC102.48 (FE)
- removed net FE-: IC101.22 (MIRR), IC102.6 (FE-)
- removed net FE0: IC101.28 (FOK), IC102.5 (FEO)
- removed net SL+: C105.1, IC102.11 (TAO), IC102.13 (SL+), P5.1 (Pin_1)
- removed net TGU: IC101.21 (DEFECT), IC102.8 (TGU)
- new net: C138.1, C138.2, IC102.36 (FSW), R105.1
- new net: C138.2, IC102.15 (SL-), R105.1, R105.1
- new net: C105.1, R105.2
- new net: C105.2, R105.1
- new net: IC102.30 (VCOF), R105.2
- new net: C138.2, IC102.32 (C864)
- new net MDP: IC102.34 (MDP)
- new net MDS: R105.2
- new net PDI: C138.1, IC102.28 (PDI), R105.2
- new net PDO: R105.1, R105.1
- new net SLO: C138.1, IC102.14 (SLO), R105.2, R105.2
- new net TAO: C105.1, IC102.11 (TAO), R105.1, R105.1, R105.2
- new net VCOI: C138.1, R105.2
- new net VCOO: R105.1
- new net XLT: IC102.24 (XLT), R105.1
- no-connect marks 0 -> 1
Other:
- moved on the sheet: C105, IC1, IC102, IC107A, IC107B, IC107C, P2, P3, P5, R105

Commit message: More passives, custom footprints, etc.
Parts:
- C105: footprint A-PCENGINE:Elec_P5.00mm -> A-PCENGINE:Elec_P5.00mm_D7mm
- IC107, IC202, IC203: footprint Package_SO:SO-8_5.3x6.2mm_P1.27mm -> A-PCENGINE:SO-8_P1.27mm
- IC201: footprint Package_SO:SO-20_5.3x12.6mm_P1.27mm -> A-PCENGINE:SO-20_P1.27mm_Gutters
Connections:
- net +9V: now also IC107.8 (V+)
- no-connect marks 1 -> 2
Changed lines of the file:
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@@
   (junction (at 273.685 44.45) (diameter 0) (color 0 0 0 0)
   )
+  (no_connect (at 81.28 78.74))
   (no_connect (at -56.515 178.435))
   (wire (pts (xy 264.795 71.12) (xy 267.97 71.12))
@@
       (effects (font (size 1.27 1.27)))
     )
-    (property "Footprint" "Package_SO:SO-8_5.3x6.2mm_P1.27mm" (at 294.005 244.475 0)
+    (property "Footprint" "A-PCENGINE:SO-8_P1.27mm" (at 294.005 244.475 0)
       (effects (font (size 1.27 1.27)) hide)
     )
@@
       (effects (font (size 1.27 1.27)))
     )
-    (property "Footprint" "Package_SO:SO-8_5.3x6.2mm_P1.27mm" (at 190.5 78.74 0)
+    (property "Footprint" "A-PCENGINE:SO-8_P1.27mm" (at 190.5 78.74 0)
       (effects (font (size 1.27 1.27)) hide)
     )
@@
       (effects (font (size 1.27 1.27)))
     )
-    (property "Footprint" "Package_SO:SO-8_5.3x6.2mm_P1.27mm" (at 341.63 132.715 0)
+    (property "Footprint" "A-PCENGINE:SO-8_P1.27mm" (at 341.63 132.715 0)
       (effects (font (size 1.27 1.27)) hide)
     )
@@
       (effects (font (size 1.27 1.27)) (justify left))
     )
-    (property "Footprint" "Package_SO:SO-8_5.3x6.2mm_P1.27mm" (at 269.24 226.695 0)
+    (property "Footprint" "A-PCENGINE:SO-8_P1.27mm" (at 269.24 226.695 0)
       (effects (font (size 1.27 1.27)) hide)
     )
@@
       (effects (font (size 1.27 1.27)) (justify left))
     )
-    (property "Footprint" "A-PCENGINE:Elec_P5.00mm" (at 254.3048 59.69 0)
+    (property "Footprint" "A-PCENGINE:Elec_P5.00mm_D7mm" (at 254.3048 59.69 0)
       (effects (font (size 1.27 1.27)) hide)
     )
@@
       (effects (font (size 1.27 1.27)) (justify left))
     )
-    (property "Footprint" "Package_SO:SO-8_5.3x6.2mm_P1.27mm" (at 227.33 102.87 0)
+    (property "Footprint" "A-PCENGINE:SO-8_P1.27mm" (at 227.33 102.87 0)
       (effects (font (size 1.27 1.27)) hide)
     )
@@
       (effects (font (size 1.27 1.27)) (justify left))
     )
-    (property "Footprint" "A-PCENGINE:Elec_P5.00mm" (at 236.5502 245.11 0)
+    (property "Footprint" "A-PCENGINE:Elec_P5.00mm_D7mm" (at 236.5502 245.11 0)
       (effects (font (size 1.27 1.27)) hide)
     )
@@
       (effects (font (size 1.27 1.27)))
     )
-    (property "Footprint" "Package_SO:SO-8_5.3x6.2mm_P1.27mm" (at 190.5 60.96 0)
+    (property "Footprint" "A-PCENGINE:SO-8_P1.27mm" (at 190.5 60.96 0)
       (effects (font (size 1.27 1.27)) hide)
     )
@@
       (effects (font (size 1.27 1.27)))
     )
-    (property "Footprint" "Package_SO:SO-8_5.3x6.2mm_P1.27mm" (at 224.79 62.23 0)
+    (property "Footprint" "A-PCENGINE:SO-8_P1.27mm" (at 224.79 62.23 0)
       (effects (font (size 1.27 1.27)) hide)
     )
@@
     )
   )
+  (symbol (lib_id "power:+9V") (at 266.7 210.185 0) (unit 1)
+    (in_bom yes) (on_board yes) (dnp no) (fields_autoplaced)
+    (property "Reference" "#PWR030" (at 266.7 213.995 0)
+      (effects (font (size 1.27 1.27)) hide)
+    )
+    (property "Value" "+9V" (at 266.7 206.375 0)
+      (effects (font (size 1.27 1.27)))
+    )
+    (property "Footprint" "" (at 266.7 210.185 0)
+      (effects (font (size 1.27 1.27)) hide)
+    )
+    (property "Datasheet" "" (at 266.7 210.185 0)
+      (effects (font (size 1.27 1.27)) hide)
+    )
+    (pin "1")
+    (instances
+      (project "PCE"
+        (path "/c1c718c6-a427-431e-a18b-e46f94ae8e09/ba362b1f-3cb7-4861-9385-2b05dca17551"
+          (reference "#PWR030") (unit 1)
+        )
+        (path "/c1c718c6-a427-431e-a18b-e46f94ae8e09/bb2f9872-1813-43e0-bcfc-5c5426bf43ce"
+          (reference "#PWR0136") (unit 1)
+        )
+      )
+    )
+  )
   (symbol (lib_id "Device:R") (at 339.09 146.05 0) (mirror y) (unit 1)
     (in_bom yes) (on_board yes) (dnp no)
@@
       (effects (font (size 1.27 1.27)) (justify left))
     )
-    (property "Footprint" "Package_SO:SO-20_5.3x12.6mm_P1.27mm" (at 349.25 182.88 0)
+    (property "Footprint" "A-PCENGINE:SO-20_P1.27mm_Gutters" (at 349.25 182.88 0)
       (effects (font (size 1.27 1.27)) hide)
     )
@@
       (effects (font (size 1.27 1.27)))
     )
-    (property "Footprint" "Package_SO:SO-8_5.3x6.2mm_P1.27mm" (at 224.79 80.01 0)
+    (property "Footprint" "A-PCENGINE:SO-8_P1.27mm" (at 224.79 80.01 0)
       (effects (font (size 1.27 1.27)) hide)
     )
@@
       (effects (font (size 1.27 1.27)) (justify left))
     )
-    (property "Footprint" "Package_SO:SO-8_5.3x6.2mm_P1.27mm" (at 214.63 102.87 0)
+    (property "Footprint" "A-PCENGINE:SO-8_P1.27mm" (at 214.63 102.87 0)
       (effects (font (size 1.27 1.27)) hide)
     )

Commit message: Top layer first draft.
Parts:
- added C105 (x9): ?, A-PCENGINE:SMD_0805_Narrow, symbol Device:C
- added C105 (x4): ~, A-PCENGINE:CP_8x2mm, symbol Device:C_Polarized
- added C105 (x4): ~, A-PCENGINE:CP_6x1.5mm, symbol Device:C_Polarized
- added C105: ?, A-PCENGINE:SMD_2010, symbol Device:C
- added P3: ~, A-PCENGINE:Header_1x02_P2.00mm, symbol Connector_Generic:Conn_01x02
- added R105 (x14): ?, A-PCENGINE:SMD_0805_Narrow, symbol Device:R
- added R105: ?, A-PCENGINE:SMD_0805_Narrow_Long, symbol Device:R
- added VR101, VR102, VR103, VR104, VR105: ~, A-PCENGINE:Duo_VR, symbol Device:R_Potentiometer
- P1, P2: footprint Connector_PinHeader_2.00mm:PinHeader_1x08_P2.00mm_Vertical -> A-PCENGINE:Header_1x08_P2.00mm
- P3: footprint Connector_PinHeader_2.00mm:PinHeader_1x07_P2.00mm_Vertical -> A-PCENGINE:Header_1x07_P2.00mm_Wide
- P5: footprint Connector_PinHeader_2.00mm:PinHeader_1x06_P2.00mm_Vertical -> A-PCENGINE:Header_1x06_P2.00mm
- renumbered IC1 to IC109
Connections:
- net +5VD: now also C105.1, C105.1, R105.2
- net ATSC: now also IC101.14 (VR), IC101.9 (VC), C105.1, C105.1, C105.1, C105.2, C105.2, C105.2, R105.2, R105.2, VR104.1
- net DATA: now also IC201.8 (DATA)
- net FE: now also VR104.2
- net GND: now also C105.2, R105.1, C105.1, C105.2, C105.2, R105.2
- net GNDA: now also C105.2, C105.2, C105.2, R105.1
- net at C105.2, IC102.13 (SL+), R105.2: now also C105.1
- net at IC109.10 (OUTA1), P2.6 (Pin_6): now also P3.1 (Pin_1)
- net at C105.1, IC109.2 (OUT0), IC109.4 (INA0)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: now also P3.2 (Pin_2)
- net RFO: now reaches IC101.2 (RFO), P5.2 (Pin_2), TP10.1
- net RFO: now also C105.2, C105.2, R105.2
- net at IC101.29 (~{LD_ON}), P5.4 (Pin_4), TP11.1: now also R105.2
- net at P5.5 (Pin_5), R105.1: now also C105.1
- net RFI: now reaches IC101.1 (RFI)
- net RFI: now also C105.1
- net EO: now reaches IC101.12 (EO)
- net EO: now also VR101.1
- net EI: now reaches IC101.13 (EI)
- net EI: now also VR101.2
- net CC2: now reaches IC101.15 (CC2)
- net CC2: now also C105.2
- net CC1: now reaches IC101.16 (CC1)
- net CC1: now also C105.1
- net FE_BIAS: now reaches IC101.18 (FE_BIAS)
- net FE_BIAS: now also VR102.2
- net at IC101.23 (CP): now also C105.2
- net at IC101.24 (CB): now also C105.2
- net RF-: now reaches IC101.3 (RF-)
- net RF-: now also C105.1, R105.2
- net at IC101.5 (LD): now also C105.2
- net at R105.2: now also C105.1, VR104.3
- net at P2.4 (Pin_4): now also R105.2
- net at IC102.31 (3.5V), R105.1: now also C105.2, VR105.2, VR105.3
- net at IC203.1: now also C105.1, R105.1, R105.1
- net at IC203.2 (-): now also C105.2, R105.2
- net PWR1: now reaches IC201.14 (IF)
- net PWR1: now also IC201.3 (VREFH2), IC201.4 (VDD), C105.1, R105.1
- net at IC201.16 (VREFL1): now also C105.1
- net at IC201.2 (VREFH1): now also C105.1, R105.2
- net at IC203.6 (-): now also C105.2, R105.1
- net at IC203.7: now also C105.1, R105.1, R105.1
- net at R105.1: now also VR105.1
- net at P1.6 (Pin_6): now also C105.1
- new net: R105.1, VR102.1
- new net: R105.1, VR102.3
- new net: C105.2, R105.1
- new net: R105.2, R105.2
- new net: R105.1, R105.2
- new net: R105.1, R105.1
- new net: R105.1, VR101.3
- new net ACTIVE: R105.1
- new net X: R105.2
- new net Y: R105.2
Other:
- moved on the sheet: C138, IC203A, IC203B, P2, R105
