File: cd_rom_mech.kicad_sch (KiCad schematic)
At the start: 122 parts, among them IC101 CXA1081, IC102 CXA1082BQ, IC107 RC4558, IC109 BA6290A, IC2 BA6290A, IC201 LC7881M, IC202 RC4558, IC203 RC4558, P1 Conn_01x08, P2 Conn_01x08, P3 Conn_01x07, P5 Conn_01x05

Commit message: More passives on back.
Parts:
- added C105 (x2): ~, A-PCENGINE:CP_1206, symbol Device:C_Polarized
- added C105 (x3): ~, A-PCENGINE:CP_2010, symbol Device:C_Polarized
- added C138: ?, A-PCENGINE:SMD_0805_Narrow_Long, symbol Device:C
- added D501: D, A-PCENGINE:Transistor_SMD, symbol Device:D
- added IC304: ?, A-PCENGINE:SOT-89-3, symbol Connector_Generic:Conn_01x03
- added L106: ~, A-PCENGINE:SMD_1210, symbol Device:L
- added L106: ~, A-PCENGINE:SMD_0805_Narrow_Long, symbol Device:L
- added R105 (x5): ?, A-PCENGINE:SMD_0805_Narrow_Long, symbol Device:R
- added R105: ?, A-PCENGINE:SMD_1210, symbol Device:R
- added TP35, TP36, TP37, TP38, TP39, TP40: ~, A-PCENGINE:Test_Point_1.5mm, symbol Connector:TestPoint
Connections:
- net +5VD: now also IC102.10 (AVCC), C105.1, C105.1, C105.1, C138.2, L106.1, L106.2, R105.1, R105.2, R105.2
- net ATSC: now also C105.1, C105.2, R105.1
- net GND: now also IC101.25 (DGND), P5.6 (Pin_6), C105.2, C105.2, C105.2, C105.2
- net GNDA: now also D501.2 (A)
- net PD: now also TP38.1
- net PWR1: now also IC201.10 (VDD)
- net at C105.1, C105.2, IC102.13 (SL+)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: now also R105.2
- net at C105.2, IC109.11 (OUT1), IC109.9 (INA1)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: now also TP39.1
- net at IC101.20 (TE), P5.3 (Pin_3): now also R105.2
- net at C105.1, P5.5 (Pin_5), R105.1: now also R105.2
- net at IC101.11 (E), P1.8 (Pin_8): now also TP36.1
- net at IC101.26 (ASY): now also C105.1, R105.1
- net LD: now reaches C105.2, IC101.5 (LD)
- net LD: now also IC304.1 (Pin_1)
- net TZCC: now reaches C105.2
- net TZCC: now also R105.1
- net at P2.2 (Pin_2): now also D501.1 (K), L106.2, TP37.1
- net at C105.1, P1.6 (Pin_6): now also R105.2, TP35.1
- net FSET: now reaches IC102.17 (FSET)
- net FSET: now also C138.1, R105.1
- new net: IC304.2 (Pin_2), L106.1
- new net: IC304.3 (Pin_3), R105.1
Other:
- moved on the sheet: C105, P1, R105

Commit message: Yet more passives on back.
Parts:
- added C105 (x11): ?, A-PCENGINE:SMD_0805_Narrow_Long, symbol Device:C
- added C105: ?, A-PCENGINE:SMD_0805_Narrow, symbol Device:C
- added C105: ?, A-PCENGINE:SMD_0805_Narrow_NoSilk, symbol Device:C
- added Q608 (x2): BR 29, A-PCENGINE:Transistor_SMD, symbol Device:Q_NPN_CBE
- added R105 (x14): ?, A-PCENGINE:SMD_0805_Narrow_Long, symbol Device:R
- added R105: ?, A-PCENGINE:SMD_0805_Narrow_NoSilk, symbol Device:R
- added R105 (x2): ?, A-PCENGINE:SMD_0805_Narrow, symbol Device:R
- added TP53: ~, A-PCENGINE:Test_Point_1.5mm, symbol Connector:TestPoint
Connections:
- net GNDA: now also C105.1, C105.1, C105.1, C105.1, C105.1, C105.1, C105.2, C105.2, Q608.3 (E), Q608.3 (E), R105.1, R105.1, R105.2, R105.2
- net PWR1: now also R105.2, R105.2
- net X: now also R105.2
- net Y: now also R105.2
- net at IC202.5 (+): now also C105.2, R105.1
- net at IC202.6 (-), IC202.7: now also C105.2
- net at R105.2, R105.2: now also C105.1, R105.1
- net at IC202.1, IC202.2 (-): now also C105.2
- net at IC202.3 (+): now also C105.2, R105.1
- net at R105.1, R105.2: now also C105.1, R105.1
- net at IC203.3 (+): now also C105.2, R105.1, R105.1
- net at C105.1, IC201.2 (VREFH1), R105.2: now also TP53.1
- net at IC201.1 (CH1OUT): now also R105.2
- net at IC201.20 (CH2OUT): now also R105.2
- net at IC203.5 (+): now also C105.2, R105.1, R105.1
- net at R105.1, R105.1: now also R105.1
- new net: C105.1, Q608.1 (C), R105.2 (x2)
- new net: C105.1, R105.2 (x3)
- new net: Q608.2 (B), R105.1 (x2)
- new net: C105.2, R105.1, R105.2 (x2)
- new net: C105.2, R105.1 (x2)
- new net GROOVE: R105.2, R105.2
- no-connect marks 2 -> 3
Other:
- moved on the sheet: C105, IC202A, IC202B, IC203A, IC203B, R105

Commit message: First draft complete.
Connections:
- net at TP40.1: now also C105.1, IC109.2 (OUT0), IC109.4 (INA0), P2.7 (Pin_7), P3.2 (Pin_2), R105.2
Changed lines of the file:
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@@
   (junction (at 294.005 208.28) (diameter 0) (color 0 0 0 0)
+  )
+  (junction (at 452.755 140.335) (diameter 0) (color 0 0 0 0)
   )
   (junction (at 283.845 62.23) (diameter 0) (color 0 0 0 0)
@@
     (stroke (width 0) (type default))
   )
-  (wire (pts (xy 461.645 140.335) (xy 429.26 140.335))
+  (wire (pts (xy 461.645 140.335) (xy 452.755 140.335))
     (stroke (width 0) (type default))
   )
@@
     (stroke (width 0) (type default))
   )
+  (wire (pts (xy 452.755 140.335) (xy 429.26 140.335))
+    (stroke (width 0) (type default))
+  )
   (wire (pts (xy 66.675 83.82) (xy 66.675 92.71))
     (stroke (width 0) (type default))
@@
     (stroke (width 0) (type default))
   )
+  (wire (pts (xy 452.755 140.335) (xy 452.755 148.59))
+    (stroke (width 0) (type default))
+  )

Commit message: Fix DRC errors.
Parts:
- added C105: ?, A-PCENGINE:SMD_0805_Narrow, symbol Device:C
- added TP67, TP68: ~, A-PCENGINE:Test_Point_1.5mm_THT_NoSilk, symbol Connector:TestPoint
- IC108: renamed from IC2; footprint Connector_PinSocket_2.54mm:PinSocket_1x12_P2.54mm_Vertical -> A-PCENGINE:SIL-12_P2.54mm
- IC109: footprint Connector_PinSocket_2.54mm:PinSocket_1x12_P2.54mm_Vertical -> A-PCENGINE:SIL-12_P2.54mm
Connections:
- net +5VD: now also R105.2, R105.2, R105.2
- net ATSC: now also VR103.1, C105.1
- net DATA: no longer IC201.8 (DATA)
- net GND: now also IC102.43 (DVEE); no longer C105.2, IC102.7 (SRCH)
- net PDO: now also R105.2
- net TE: now also VR103.2
- net TZCC: now also VR103.3, C105.2
- net at C105.1, R105.2: now also TP68.1
- net BW: now reaches C127.2
- net at C105.1, R105.2: now also TP67.1
- new net: C105.2, IC102.7 (SRCH)
- new net DATA2: IC201.8 (DATA)
Other:
- moved on the sheet: C105, R105, VR103

Commit message: General clean-up.
Parts:
- added TP65, TP69: ~, A-PCENGINE:Test_Point_1.5mm, symbol Connector:TestPoint
- C138: footprint A-PCENGINE:SMD_1206 -> A-PCENGINE:CP_1206; symbol Device:C -> Device:C_Polarized
- renumbered TP1 to TP101
Connections:
- net ATSC: now also TP65.1
- net GND: now also TP69.1
Other:
- moved on the sheet: TP11

Commit message: Add resistor values to schematics.
Parts:
- C105, R105: value ? -> N/P
- IC304: value ? -> No Markings; symbol Connector_Generic:Conn_01x03 -> Device:Q_PNP_CBE
- R105: value ? -> 10K
- R105: value ? -> 220K
- R105: value ? -> 75K
- R105: value ? -> 10M
- R105: value ? -> 100K
- R105: value ? -> 4.7K
- R105: value ? -> 10K 1%
- R105: value ? -> 47K
- R105: value ? -> 1K
- R105: value ? -> 6.8K
- R105: value ? -> 120K
- R105: value ? -> 390
- R105: value ? -> 5.1K
- R105: value ? -> 15K
- R105: value ? -> 2.2K
- R105: value ? -> 24K
- R105: value ? -> 15K?
- R105: value ? -> 3.3K
- R105: value ? -> 180K
- R105: value ? -> 1.8K
- R105: value ? -> 22
- R105: value ? -> 12K
- R105: value ? -> 20K
- R105: value ? -> 91K
- R105: value ? -> 22K
- R105: value ? -> 680
- R105: value ? -> 510K
- R105: value ? -> 9.4K
Connections:
- no-connect marks 3 -> 4
Other:
- note added: "10K + 160K in parralel"
- moved on the sheet: C105, D501, L106, P2, R105, TP37, TP38, TP39, TP40

Commit message: Schematic clean-up.
Connections:
- net DVCC renamed DCLK
Changed lines of the file:
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@@
     )
   )
-  (global_label "DVCC" (shape input) (at -54.61 188.595 0) (fields_autoplaced)
+  (global_label "DCLK" (shape input) (at -54.61 188.595 0) (fields_autoplaced)
     (effects (font (size 1.27 1.27)) (justify left))
-    (property "Intersheetrefs" "${INTERSHEET_REFS}" (at -46.7262 188.595 0)
+    (property "Intersheetrefs" "${INTERSHEET_REFS}" (at -46.7867 188.595 0)
       (effects (font (size 1.27 1.27)) (justify left) hide)
     )

Commit message: Schematic clean-up (IFU ASIC and other stuff).
Connections:
- no-connect marks 4 -> 6
Other:
- moved on the sheet: C105, D501, IC107A, IC107B, IC107C, IC108, IC109, IC201, IC202A, IC202B, IC202C, IC203A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
