File: interface.kicad_sch (KiCad schematic)
At the start: 20 parts, among them IC107 RC4558, IC501 D91317GD, IC502 MSM5205, IC503 RC4558, IC504 4053, IC521 RC4558

Commit message: More passives, custom footprints, etc.
Parts:
- added C105 (x14): ?, A-PCENGINE:SMD_0805_Narrow, symbol Device:C
- added C105 (x3): ?, A-PCENGINE:CP_8x2mm, symbol Device:C_Polarized
- added C105 (x6): ?, A-PCENGINE:SMD_0805_Narrow_Long, symbol Device:C
- added C105 (x9): ?, A-PCENGINE:CP_6x1.5mm, symbol Device:C_Polarized
- added C105: ?, A-PCENGINE:CP_8.4x1.7mm, symbol Device:C_Polarized
- added C105 (x5): ?, A-PCENGINE:CP_7x2mm, symbol Device:C_Polarized
- added C105: N/P, A-PCENGINE:SMD_0805_Narrow, symbol Device:C
- added C105 (x2): N/P, A-PCENGINE:SMD_0805_Narrow_Long, symbol Device:C
- added C113: ~, A-PCENGINE:CP_8x2mm, symbol Device:C_Polarized
- added C113: ~, A-PCENGINE:Elec_P5.00mm_D12mm_Pad3mm, symbol Device:C_Polarized
- added D601: P, A-PCENGINE:Transistor_SMD, symbol Device:D_Dual_CommonAnode_KKA
- added J1: Conn_01x05, A-PCENGINE:Duo_Dial_5P, symbol Connector_Generic:Conn_01x05
- added R905 (x27): ?, A-PCENGINE:SMD_0805_Narrow, symbol Device:R
- added TP7: ~, A-PCENGINE:Test_Point_1.5mm, symbol Connector:TestPoint
- added X601: ~, A-PCENGINE:Crystal_5x10mm, symbol Device:Crystal_GND2
- C105: footprint A-PCENGINE:SMD_0805_Narrow -> A-PCENGINE:SMD_0805_Narrow_Long
- IC107: footprint Package_SO:SO-8_5.3x6.2mm_P1.27mm -> A-PCENGINE:SO-8_P1.27mm
- IC503, IC521: footprint Package_SO:SO-8_5.3x6.2mm_P1.27mm -> A-PCENGINE:SO-8_P1.27mm_Gutters
- IC504: footprint Package_SO:SOIC-16_4.55x10.3mm_P1.27mm -> A-PCENGINE:SO-16_P1.27mm_Gutters
Connections:
- net +5V is gone; now on net +5VD: L106.2, R105.2, RA511.5 (R4.2), RA511.6 (R3.2), RA511.7 (R2.2), RA511.8 (R1.2), RA512.5 (R4.2), RA512.6 (R3.2), RA512.7 (R2.2), RA512.8 (R1.2), RA513.5 (R4.2), RA513.6 (R3.2), RA513.7 (R2.2), RA513.8 (R1.2)
- net +5VD: now also C105.2, C105.2, R905.2
- net +5VP: now also C105.2, C105.2, C113.1, R905.2
- net GND: now also C105.1, C105.1, C105.1, C105.1, C105.1, C105.1, C105.1, C105.1, C105.1, C105.1, C105.1, C105.1, C105.1, C105.2, C105.2, C105.2, C113.2, R905.2, X601.2; no longer IC502.12 (T1), IC502.2 (S2), IC502.9 (VSS)
- net GNDA: now also IC502.12 (T1), IC502.2 (S2), IC502.9 (VSS), IC504.6 (Inh), IC504.7 (VEE), IC504.8 (VSS), C105.1, C105.1, C105.1, C105.2, C105.2, C105.2, C105.2, C105.2, C105.2, C105.2, C105.2, C113.2, J1.1 (Pin_1), J1.2 (Pin_2), J1.3 (Pin_3), R905.1, R905.2
- net VCC_501: now reaches IC501.1, IC501.14, IC501.26, IC501.30, IC501.61, IC501.90, L106.1
- net VCC_501: now also C105.1, C105.2, C105.2, C105.2, C105.2, C105.2, C105.2, C105.2, C105.2, C105.2, C105.2, R905.2
- net at IC501.74: now also R905.1
- net at IC501.79: now also R905.1
- net at IC501.83: now also C105.1, X601.1
- net at IC501.84: now also C105.1, X601.3
- net at IC501.94: now also C105.2, TP7.1
- net at IC107.5 (+): now also R905.1
- net at IC107.7: now also R905.1
- net at IC3.10 (VOL2): now also R905.1, R905.2
- net at IC3.12 (MODE), IC3.4 (VREF): now also R905.1
- net at IC3.13 (OUT2): now also C105.2
- net at IC3.14 (IN2): now also C105.1
- net at IC3.2 (IN1): now also C105.1
- net at IC3.3 (OUT1): now also C105.2
- net at IC3.5 (FILTER): now also C105.1
- net at IC3.8 (VOL1): now also C105.1
- net at IC503.3 (+), IC503.5 (+): now also IC521.3 (+), IC521.5 (+), C105.1, R905.1, R905.2
- net at IC503.6 (-): now also R905.2
- net at IC503.7: now also C105.2, R905.1
- net at IC107.3 (+), IC107.5 (+): now also C105.1, C105.1
- net at IC107.6 (-): now also R905.1
- net at IC107.7: now also C105.1
- net at IC521.6 (-): now also R905.2, R905.2, R905.2
- net at IC521.7: now also C105.2, R905.1
- net at IC503.1: now also IC504.4 (Z), C105.1, R905.2
- net at IC503.2 (-): now also C105.2, R905.2
- net at IC504.1 (Y1): now also R905.2
- net at IC504.12 (X0): now also R905.2
- net at IC504.13 (X1): now also R905.2
- net at IC504.2 (Y0): now also R905.1
- net at IC504.3 (Z1): now also R905.1, R905.2
- net at IC502.1 (S1), IC502.18 (VDD), IC502.3 (4B/~{3B}): now also C105.1, R905.1
- net at IC521.1: now also C105.2, R905.1
- net at IC521.2 (-): now also R905.1, R905.1, R905.2
- net at IC107.1: now also R905.1, R905.1
- net at IC107.2 (-): now also R905.2
- net at IC107.1: now also C105.1, R905.1
- net at IC107.2 (-): now also R905.1, R905.2
- new net: C105.2, R905.1, R905.1, R905.1
- new net: C105.1, R905.2 (x4)
- new net: C105.2, J1.5 (Pin_5), R905.1
- new net: C105.2, J1.4 (Pin_4), R905.1
- new net: D601.2 (K), R905.1
- new net AGND: C105.2
- new net AUDIO-C: C105.1, C105.1
Other:
- moved on the sheet: IC107A, IC107B, IC107C, IC503A, IC503B, IC503C, IC504, IC521A, IC521B, IC521C, RA501, RA502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

Commit message: Top layer first draft.
Parts:
- removed C113: ~, A-PCENGINE:Elec_P5.00mm_D12mm_Pad3mm, symbol Device:C_Polarized
- added JK602: Audio, A-PCENGINE:Duo_Audio_Jack, symbol Connector_Audio:AudioJack3
- added L106 (x2): ~, A-PCENGINE:SMD_1206_C, symbol Device:L
- added L106: N/P, A-PCENGINE:SMD_1206_C_NoSilk, symbol Device:L
- added R905: N/P, A-PCENGINE:SMD_0805_Narrow_Long_NoSilk, symbol Device:R
- IC502: footprint Package_DIP:DIP-18_W7.62mm -> A-PCENGINE:DIP-18_W
- RA501, RA502, RA503, RA504, RA511, RA512, RA513: footprint Resistor_SMD:R_Array_Concave_4x0603 -> A-PCENGINE:R_Array_4x0603
- renumbered J1 to VR601
Connections:
- net GNDA: now also JK602.S, L106.1, L106.2, R905.1, R905.2
- net BUCKAROO: now reaches C105.2, IC501.94, TP7.1
- net X: now reaches IC504.14 (X)
- net Y: now reaches IC504.15 (Y)
- new net: JK602.T, L106.2
- new net: JK602.R, L106.2
Other:
- moved on the sheet: TP7
