File: interface.kicad_sch (KiCad schematic)
At the start: 98 parts, among them IC107 RC4558, IC501 D91317GD, IC502 MSM5205, IC503 RC4558, IC504 4053, IC521 RC4558

Commit message: More passives on back.
Parts:
- added C105 (x8): ?, A-PCENGINE:SMD_0805_Narrow_Long, symbol Device:C
- added D602: P 32, A-PCENGINE:Transistor_SMD, symbol Device:D_Dual_CommonAnode_AKK
- added Q608, Q609: AAR 29, A-PCENGINE:Transistor_SMD, symbol Device:Q_NPN_CBE
- added R105 (x11), R905 (x4): ?, A-PCENGINE:SMD_0805_Narrow_Long, symbol Device:R
- added R905: ?, A-PCENGINE:SMD_0805_Narrow, symbol Device:R
- added TP1 (x2): ~, A-PCENGINE:Test_Point_1.5mm, symbol Connector:TestPoint
Connections:
- net +5VP: now also R105.1, R105.2
- net ABC: now also TP1.1
- net GNDA: now also C105.1, C105.1, C105.1, C105.1, C105.1, C105.2, C105.2, C105.2, Q608.3 (E), Q609.3 (E), R105.1, R105.2, R905.2, R905.2
- net at C105.1, IC502.1 (S1), IC502.18 (VDD)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: now also C105.1
- net at C105.2: now also JK602.R, L106.1, L106.2, C105.2, Q609.1 (C), R905.1
- net at C105.2: now also JK602.T, L106.1, L106.2, C105.2, Q608.1 (C), R905.1
- net at IC107.7, R905.1: now also R905.1
- net at IC107.2 (-), R905.2: now also R105.2
- net at IC107.5 (+), R905.1: now also C105.1
- net at IC107.6 (-): now also R105.1, R905.2
- net at C105.1: now also R105.1, R105.1
- net at C105.1, R905.2: now also R105.1
- net at C105.1: now also R105.1
- net at D601.1 (K): now also D602.1 (A)
- net at IC503.6 (-), R905.2: now also R105.1
- net at C105.1: now also R105.2
- net at IC107.3 (+): now also C105.2, R105.2
- net at C105.2: now also R105.1
- new net: C105.2, R105.2, R105.2, TP1.1
- new net: C105.1, R105.1, R105.1, R105.2
- new net: D602.2 (K), R905.2
- new net: D602.3 (K), R905.2
- new net: C105.2, R105.2, R105.2, R105.2
- new net: Q609.2 (B), R905.1
- new net: Q608.2 (B), R905.1
Other:
- moved on the sheet: C105, D601, IC107A, IC502, JK602, L106, R905

Commit message: Yet more passives on back.
Parts:
- added Q102: 26, A-PCENGINE:Transistor_SMD, symbol Device:Q_NPN_CBE
- added R105 (x2): ?, A-PCENGINE:SMD_0805_Narrow_Long, symbol Device:R
- added TP1 (x2): ~, A-PCENGINE:Test_Point_1.5mm, symbol Connector:TestPoint
Connections:
- net BUCKAROO: now also R105.1
- net GND: now also Q102.3 (E)
- net RAMBO: now reaches IC501.49
- net at IC501.78: now also Q102.2 (B), TP1.1
- net PWR2: now reaches D601.1 (K), D602.1 (A)
- new net: Q102.1 (C), R105.2, R105.2, TP1.1
- new net DX: R105.1

Commit message: First draft complete.
Parts:
- added C105 (x4): ?, A-PCENGINE:SMD_0805_Narrow_Long, symbol Device:C
- added C105: ?, A-PCENGINE:SMD_0805_Narrow, symbol Device:C
- added Q1 (x3): ~, A-PCENGINE:Transistor_SMD, symbol Device:Q_NPN_CBE
- added Q606: 15, A-PCENGINE:Transistor_SMD, symbol Device:Q_PNP_CBE
- added R105 (x4), R905 (x15): ?, A-PCENGINE:SMD_0805_Narrow_Long, symbol Device:R
- added R905 (x3): ?, A-PCENGINE:SMD_0805_Narrow, symbol Device:R
- added TP40 (x7): ~, A-PCENGINE:Test_Point_1.5mm, symbol Connector:TestPoint
- D601: symbol Device:D_Dual_CommonAnode_KKA -> Device:D_Dual_CommonAnode_AKK
Connections:
- net +5VD: now also Q606.3 (E); no longer C105.2
- net +5VP: now also C105.1, R905.2
- net GND: now also Q1.3 (E), R105.2
- net GNDA: now also C105.2, C105.2, C105.2, Q1.3 (E), Q1.3 (E), R905.1, R905.2, R905.2; no longer C105.1, C105.1, Q608.3 (E), Q609.3 (E), R905.2, R905.2
- net P79: now reaches IC501.79, R905.1
- net P79: now also Q606.2 (B), TP40.1
- net P80: now reaches IC501.80
- net P80: now also R105.1
- net at C105.1, IC503.3 (+), IC503.5 (+)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: now also TP40.1
- net at C105.1, C105.1, IC107.3 (+)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: now also R905.1, R905.2, TP40.1
- net at IC107.2 (-), R905.1, R905.2: now also R905.1, R905.2, R905.2, R905.2
- net at C105.2: now also R905.1, R905.2
- net at C105.1, IC3.8 (VOL1): now also R105.1, R105.2, TP40.1
- net at D601.2 (K): now also R905.1; no longer R905.1
- net at D601.3 (K): now also R905.1
- net at IC107.6 (-), R905.1: now also R905.1, R905.1, R905.1, R905.2, R905.2
- net at C105.1, IC107.7: now also R905.1
- net at C105.1: now also R905.2
- net at R905.2: now also Q1.2 (B)
- net at C105.2: now also R905.2, R905.1, R905.2
- net at IC504.5 (Z0): now also R905.1, R905.1
- net at R905.2: now also C105.2, R905.1, R905.2
- net at C105.1: now also R905.1
- new net: Q606.1 (C), R105.1
- new net: C105.1, R905.2, R905.2 (x2)
- new net: C105.1, C105.1, Q608.3 (E), Q609.3 (E), R905.2, R905.2
- new net: C105.2, R905.1, TP40.1 (x2)
- new net: Q1.1 (C), R105.1, R105.2
- new net: Q1.2 (B), R105.2, TP40.1
- new net: Q1.2 (B), R905.2
- new net +5V: C105.2
- new net AUDIO-L: C105.1
- new net AUDIO-R: C105.1
- new net DIN_L: Q1.1 (C), R905.1
- new net DIN_R: Q1.1 (C), R905.1
Other:
- moved on the sheet: C105, D601, D602, IC107A, IC107B, JK602, L106, Q608, Q609, R105, R905, VR601

Commit message: Fix DRC errors.
Parts:
- removed C105 (x2): ?, A-PCENGINE:SMD_0805_Narrow_Long, symbol Device:C
Connections:
- net GNDA: now also C105.1, C105.1, Q608.3 (E), Q609.3 (E), R905.2, R905.2
- net at D601.2 (K): now also R905.1; no longer R905.1
- net at D601.3 (K): now also R905.1; no longer R905.1
Changed lines of the file:
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@@
   (junction (at 767.715 94.615) (diameter 0) (color 0 0 0 0)
   )
-  (junction (at 46.355 82.55) (diameter 0) (color 0 0 0 0)
-  )
   (junction (at 195.58 3.175) (diameter 0) (color 0 0 0 0)
   )
@@
   (junction (at -43.815 67.945) (diameter 0) (color 0 0 0 0)
   )
-  (junction (at 60.96 42.545) (diameter 0) (color 0 0 0 0)
-  )
   (junction (at 506.73 210.185) (diameter 0) (color 0 0 0 0)
   )
@@
   (junction (at 146.05 31.115) (diameter 0) (color 0 0 0 0)
   )
+  (junction (at 683.895 108.585) (diameter 0) (color 0 0 0 0)
+  )
   (junction (at 206.375 235.585) (diameter 0) (color 0 0 0 0)
   )
@@
     (stroke (width 0) (type default))
   )
-  (wire (pts (xy 38.1 42.545) (xy 38.1 53.975))
-    (stroke (width 0) (type default))
-  )
   (wire (pts (xy 204.47 109.22) (xy 187.96 109.22))
     (stroke (width 0) (type default))
@@
     (stroke (width 0) (type default))
   )
-  (wire (pts (xy 60.96 41.275) (xy 60.96 42.545))
-    (stroke (width 0) (type default))
-  )
   (wire (pts (xy 694.055 63.5) (xy 694.055 59.69))
     (stroke (width 0) (type default))
@@
     (stroke (width 0) (type default))
   )
+  (wire (pts (xy 683.895 108.585) (xy 683.895 114.935))
+    (stroke (width 0) (type default))
+  )
   (wire (pts (xy 29.845 111.76) (xy 88.9 111.76))
     (stroke (width 0) (type default))
@@
     (stroke (width 0) (type default))
   )
-  (wire (pts (xy 38.1 42.545) (xy 60.96 42.545))
-    (stroke (width 0) (type default))
-  )
   (wire (pts (xy 38.1 106.68) (xy 47.625 106.68))
     (stroke (width 0) (type default))
@@
     (stroke (width 0) (type default))
   )
-  (wire (pts (xy 38.1 61.595) (xy 38.1 82.55))
-    (stroke (width 0) (type default))
-  )
   (wire (pts (xy 506.73 219.075) (xy 506.73 221.615))
     (stroke (width 0) (type default))
@@
     (stroke (width 0) (type default))
   )
-  (wire (pts (xy 46.355 82.55) (xy 38.1 82.55))
+  (wire (pts (xy 38.1 82.55) (xy 114.3 82.55))
     (stroke (width 0) (type default))
   )
@@
     (stroke (width 0) (type default))
   )
-  (wire (pts (xy 46.355 52.07) (xy 46.355 53.975))
-    (stroke (width 0) (type default))
-  )
   (wire (pts (xy 241.3 247.015) (xy 233.045 247.015))
     (stroke (width 0) (type default))
@@
     (stroke (width 0) (type default))
   )
-  (wire (pts (xy 46.355 61.595) (xy 46.355 82.55))
-    (stroke (width 0) (type default))
-  )
   (wire (pts (xy 300.99 219.71) (xy 300.99 226.06))
     (stroke (width 0) (type default))
@@
     (stroke (width 0) (type default))
   )
-  (wire (pts (xy 60.96 42.545) (xy 60.96 59.055))
+  (wire (pts (xy 60.96 41.275) (xy 60.96 59.055))
     (stroke (width 0) (type default))
   )
@@
     (stroke (width 0) (type default))
   )
-  (wire (pts (xy 114.3 82.55) (xy 46.355 82.55))
-    (stroke (width 0) (type default))
-  )
   (wire (pts (xy 278.13 114.935) (xy 278.13 112.395))
     (stroke (width 0) (type default))
@@
     )
   )
-  (symbol (lib_id "Device:C") (at 46.355 57.785 0) (mirror x) (unit 1)
-    (in_bom yes) (on_board yes) (dnp no)
-    (property "Reference" "C105" (at 43.18 55.245 0)
-      (effects (font (size 1.27 1.27)))
-    )
-    (property "Value" "?" (at 43.18 60.325 0)
-      (effects (font (size 1.27 1.27)))
-    )
-    (property "Footprint" "A-PCENGINE:SMD_0805_Narrow_Long" (at 47.3202 53.975 0)
-      (effects (font (size 1.27 1.27)) hide)
-    )
-    (property "Datasheet" "~" (at 46.355 57.785 0)
-      (effects (font (size 1.27 1.27)) hide)
-    )
-    (pin "1")
-    (pin "2")
-    (instances
-      (project "PCE"
-        (path "/c1c718c6-a427-431e-a18b-e46f94ae8e09/1d91d06a-381a-4a70-bfc1-2abf4d159a91"
-          (reference "C105") (unit 1)
-        )
-        (path "/c1c718c6-a427-431e-a18b-e46f94ae8e09/ed9120da-14d8-40be-9026-fb246d72bf2f"
-          (reference "C124") (unit 1)
-        )
-        (path "/c1c718c6-a427-431e-a18b-e46f94ae8e09/c78d7e8a-3e65-46f4-91f4-96eb31925bea"
-          (reference "C133") (unit 1)
-        )
-        (path "/c1c718c6-a427-431e-a18b-e46f94ae8e09/ba362b1f-3cb7-4861-9385-2b05dca17551"
-          (reference "C148") (unit 1)
-        )
-        (path "/c1c718c6-a427-431e-a18b-e46f94ae8e09/f2e7b294-149a-4ec9-8398-41569f37f2ee"
-          (reference "C508") (unit 1)
-        )
-      )
-    )
-  )
   (symbol (lib_id "Device:R") (at 268.605 201.295 0) (mirror y) (unit 1)
     (in_bom yes) (on_board yes) (dnp no)
@@
     )
   )
-  (symbol (lib_id "power:+5V") (at 46.355 52.07 0) (unit 1)
-    (in_bom yes) (on_board yes) (dnp no) (fields_autoplaced)
-    (property "Reference" "#PWR0193" (at 46.355 55.88 0)
-      (effects (font (size 1.27 1.27)) hide)
-    )
-    (property "Value" "+5V" (at 46.355 46.99 0)
-      (effects (font (size 1.27 1.27)))
-    )
-    (property "Footprint" "" (at 46.355 52.07 0)
-      (effects (font (size 1.27 1.27)) hide)
-    )
-    (property "Datasheet" "" (at 46.355 52.07 0)
-      (effects (font (size 1.27 1.27)) hide)
-    )
-    (pin "1")
-    (instances
-      (project "PCE"
-        (path "/c1c718c6-a427-431e-a18b-e46f94ae8e09/f2e7b294-149a-4ec9-8398-41569f37f2ee"
-          (reference "#PWR0193") (unit 1)
-        )
-      )
-    )
-  )
   (symbol (lib_id "Device:R") (at 608.965 28.575 180) (unit 1)
     (in_bom yes) (on_board yes) (dnp no) (fields_autoplaced)
@@
     )
   )
-  (symbol (lib_id "Device:D_Dual_CommonAnode_AKK") (at 421.005 92.075 270) (mirror x) (unit 1)
+  (symbol (lib_id "power:GNDA") (at 683.895 114.935 0) (unit 1)
+    (in_bom yes) (on_board yes) (dnp no) (fields_autoplaced)
+    (property "Reference" "#PWR0194" (at 683.895 121.285 0)
+      (effects (font (size 1.27 1.27)) hide)
+    )
+    (property "Value" "GNDA" (at 683.895 119.38 0)
+      (effects (font (size 1.27 1.27)))
+    )
+    (property "Footprint" "" (at 683.895 114.935 0)
+      (effects (font (size 1.27 1.27)) hide)
+    )
+    (property "Datasheet" "" (at 683.895 114.935 0)
+      (effects (font (size 1.27 1.27)) hide)
+    )
+    (pin "1")
+    (instances
+      (project "PCE"
+        (path "/c1c718c6-a427-431e-a18b-e46f94ae8e09/f2e7b294-149a-4ec9-8398-41569f37f2ee"
+          (reference "#PWR0194") (unit 1)
+        )
+      )
+    )
+  )
+  (symbol (lib_id "Device:D_Dual_CommonAnode_AKK") (at 421.005 92.075 270) (unit 1)
     (in_bom yes) (on_board yes) (dnp no)
-    (property "Reference" "D601" (at 424.18 93.345 90)
+    (property "Reference" "D601" (at 424.18 90.805 90)
       (effects (font (size 1.27 1.27)) (justify left))
     )
-    (property "Value" "P" (at 424.18 90.805 90)
+    (property "Value" "P" (at 424.18 93.345 90)
       (effects (font (size 1.27 1.27)) (justify left))
     )
@@
         )
       )
-    )
-  )
-  (symbol (lib_id "Device:C") (at 38.1 57.785 0) (mirror x) (unit 1)
-    (in_bom yes) (on_board yes) (dnp no)
-    (property "Reference" "C105" (at 34.925 55.245 0)
-      (effects (font (size 1.27 1.27)))
-    )
-    (property "Value" "?" (at 34.925 60.325 0)
-      (effects (font (size 1.27 1.27)))
-    )
-    (property "Footprint" "A-PCENGINE:SMD_0805_Narrow_Long" (at 39.0652 53.975 0)
-      (effects (font (size 1.27 1.27)) hide)
-    )
-    (property "Datasheet" "~" (at 38.1 57.785 0)
-      (effects (font (size 1.27 1.27)) hide)
-    )
-    (pin "1")
-    (pin "2")
-    (instances
-      (project "PCE"
-        (path "/c1c718c6-a427-431e-a18b-e46f94ae8e09/1d91d06a-381a-4a70-bfc1-2abf4d159a91"
-          (reference "C105") (unit 1)
-        )
-        (path "/c1c718c6-a427-431e-a18b-e46f94ae8e09/ed9120da-14d8-40be-9026-fb246d72bf2f"
-          (reference "C124") (unit 1)
-        )
-        (path "/c1c718c6-a427-431e-a18b-e46f94ae8e09/c78d7e8a-3e65-46f4-91f4-96eb31925bea"
-          (reference "C133") (unit 1)
-        )
-        (path "/c1c718c6-a427-431e-a18b-e46f94ae8e09/ba362b1f-3cb7-4861-9385-2b05dca17551"
-          (reference "C148") (unit 1)
-        )
-        (path "/c1c718c6-a427-431e-a18b-e46f94ae8e09/f2e7b294-149a-4ec9-8398-41569f37f2ee"
-          (reference "C506") (unit 1)
-        )
-      )

Commit message: General clean-up.
Parts:
- C105: footprint A-PCENGINE:CP_8.4x1.7mm -> A-PCENGINE:CP_8x2mm
Changed lines of the file:
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@@
-    (stroke (width 0) (type default))
-  )
-  (wire (pts (xy 214.63 95.25) (xy 224.79 95.25))
     (stroke (width 0) (type default))
   )
@@
     (property "Intersheetrefs" "${INTERSHEET_REFS}" (at 75.3919 170.18 0)
       (effects (font (size 1.27 1.27)) (justify right) hide)
-    )
-  )
-  (global_label "~{IOE}" (shape input) (at 224.79 95.25 0) (fields_autoplaced)
-    (effects (font (size 1.27 1.27)) (justify left))
-    (property "Intersheetrefs" "${INTERSHEET_REFS}" (at 230.8595 95.25 0)
-      (effects (font (size 1.27 1.27)) (justify left) hide)
     )
   )
@@
       (effects (font (size 1.27 1.27)) (justify left))
     )
-    (property "Footprint" "A-PCENGINE:CP_8.4x1.7mm" (at -56.8452 79.375 0)
-      (effects (font (size 1.27 1.27)) hide)
-    )
+    (property "Footprint" "A-PCENGINE:CP_8x2mm" (at -56.8452 79.375 0)
+      (effects (font (size 1.27 1.27)) hide)
+    )

Commit message: Add resistor values to schematics.
Parts:
- R105: value ? -> 470
- R105, R905: value ? -> 1K
- R105: value ? -> 82K
- R105: value ? -> 560
- R105, R905: value ? -> 270K
- R105, R905: value ? -> 10K
- R105: value ? -> 39K
- R105: value ? -> 100K
- R105, R905: value ? -> 8.2K
- R105, R905: value ? -> 47K
- R105, R905: value ? -> 6.8K
- R905: value ? -> 22
- R905: value ? -> 10K 1%
- R905: value ? -> 15K
- R905: value ? -> 47K?
- R905: value ? -> 120
- R905: value ? -> 33K
- R905: value ? -> 5.1K
- R905: value ? -> 2.2K
- R905: value ? -> 3K

Commit message: Schematic clean-up.
Connections:
- net DX renamed ~{URESET}
Changed lines of the file:
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@@
     )
   )
-  (global_label "DX" (shape input) (at 141.605 18.415 180) (fields_autoplaced)
+  (global_label "~{URESET}" (shape input) (at 141.605 18.415 180) (fields_autoplaced)
     (effects (font (size 1.27 1.27)) (justify right))
-    (property "Intersheetrefs" "${INTERSHEET_REFS}" (at 136.1403 18.415 0)
+    (property "Intersheetrefs" "${INTERSHEET_REFS}" (at 131.5442 18.415 0)
       (effects (font (size 1.27 1.27)) (justify right) hide)
     )

Commit message: Intermediate commit after renaming some nets.
Connections:
- net CFX10 is gone; now on net CFX0: IC501.96, RA503.4 (R4.1)
- net CFX8 is gone; now on net CFX2: IC501.98, RA503.2 (R2.1)
- net CFX9 is gone; now on net CFX1: IC501.97, RA503.3 (R3.1)
- net CFX0: no longer IC501.118, RA502.2 (R2.1)
- net CFX1: no longer IC501.117, RA501.3 (R3.1)
- net CFX2: no longer IC501.115
- net CFX3: now also IC501.99, RA503.1 (R1.1); no longer IC501.103, RA504.1 (R1.1)
- net CFX4: now also IC501.100, RA504.4 (R4.1); no longer IC501.102, RA504.2 (R2.1)
- net CFX6: now also IC501.102, RA504.2 (R2.1); no longer IC501.100, RA504.4 (R4.1)
- net CFX7: now also IC501.103, RA504.1 (R1.1); no longer IC501.99, RA503.1 (R1.1)
- new net CFS0: IC501.118, RA502.2 (R2.1)
- new net CFS1: IC501.117, RA501.3 (R3.1)
- new net CFS2: IC501.115
Other:
- moved on the sheet: RA504
