File: vdc.kicad_sch (KiCad schematic)
At the start: 9 parts, among them IC9001 M20256, IC9002 M20256, IC902 HUC6270

Commit message: Add proper scans, redo traces.
Parts:
- renumbered C130 to C904, C129 to C914
Changed lines of the file:
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@@
   (symbol (lib_id "Device:C") (at 276.86 140.97 0) (unit 1)
     (in_bom yes) (on_board yes) (dnp no)
-    (property "Reference" "C130" (at 278.13 137.16 0)
+    (property "Reference" "C904" (at 278.13 137.16 0)
       (effects (font (size 1.27 1.27)) (justify left))
     )
@@
       (project "PCE"
         (path "/c1c718c6-a427-431e-a18b-e46f94ae8e09/ed9120da-14d8-40be-9026-fb246d72bf2f"
-          (reference "C130") (unit 1)
+          (reference "C904") (unit 1)
         )
       )
@@
   (symbol (lib_id "Device:C") (at 205.74 201.93 0) (unit 1)
     (in_bom yes) (on_board yes) (dnp no) (fields_autoplaced)
-    (property "Reference" "C102" (at 209.55 201.295 0)
-      (effects (font (size 1.27 1.27)) (justify left))
-    )
-    (property "Value" "0.1uF" (at 209.55 203.835 0)
+    (property "Reference" "C102" (at 209.55 200.66 0)
+      (effects (font (size 1.27 1.27)) (justify left))
+    )
+    (property "Value" "0.1uF" (at 209.55 203.2 0)
       (effects (font (size 1.27 1.27)) (justify left))
     )
@@
         )
         (path "/c1c718c6-a427-431e-a18b-e46f94ae8e09/ed9120da-14d8-40be-9026-fb246d72bf2f"
-          (reference "C125") (unit 1)
+          (reference "C912") (unit 1)
         )
       )
@@
   (symbol (lib_id "Device:C") (at 276.86 81.28 0) (unit 1)
     (in_bom yes) (on_board yes) (dnp no)
-    (property "Reference" "C129" (at 278.13 77.47 0)
+    (property "Reference" "C914" (at 278.13 77.47 0)
       (effects (font (size 1.27 1.27)) (justify left))
     )
@@
       (project "PCE"
         (path "/c1c718c6-a427-431e-a18b-e46f94ae8e09/ed9120da-14d8-40be-9026-fb246d72bf2f"
-          (reference "C129") (unit 1)
+          (reference "C914") (unit 1)
         )
       )
@@
   (symbol (lib_id "Device:C") (at 231.14 201.93 0) (unit 1)
     (in_bom yes) (on_board yes) (dnp no)
-    (property "Reference" "C106" (at 234.95 201.295 0)
-      (effects (font (size 1.27 1.27)) (justify left))
-    )
-    (property "Value" "0.1uF" (at 234.95 203.835 0)
+    (property "Reference" "C106" (at 234.95 200.66 0)
+      (effects (font (size 1.27 1.27)) (justify left))
+    )
+    (property "Value" "0.1uF" (at 234.95 203.2 0)
       (effects (font (size 1.27 1.27)) (justify left))
     )
@@
         )
         (path "/c1c718c6-a427-431e-a18b-e46f94ae8e09/ed9120da-14d8-40be-9026-fb246d72bf2f"
-          (reference "C127") (unit 1)
+          (reference "C932") (unit 1)
         )
       )
@@
         )
         (path "/c1c718c6-a427-431e-a18b-e46f94ae8e09/ed9120da-14d8-40be-9026-fb246d72bf2f"
-          (reference "C124") (unit 1)
+          (reference "C902") (unit 1)
         )
       )
@@
   (symbol (lib_id "Device:C") (at 218.44 201.93 0) (unit 1)
     (in_bom yes) (on_board yes) (dnp no) (fields_autoplaced)
-    (property "Reference" "C102" (at 222.25 201.295 0)
-      (effects (font (size 1.27 1.27)) (justify left))
-    )
-    (property "Value" "0.1uF" (at 222.25 203.835 0)
+    (property "Reference" "C102" (at 222.25 200.66 0)
+      (effects (font (size 1.27 1.27)) (justify left))
+    )
+    (property "Value" "0.1uF" (at 222.25 203.2 0)
       (effects (font (size 1.27 1.27)) (justify left))
     )
@@
         )
         (path "/c1c718c6-a427-431e-a18b-e46f94ae8e09/ed9120da-14d8-40be-9026-fb246d72bf2f"
-          (reference "C126") (unit 1)
-        )
-      )
+          (reference "C922") (unit 1)
+        )
+      )

Commit message: IC routing mostly complete, start adding passives.
Parts:
- C102, C104, C106, C904, C914: footprint Capacitor_SMD:C_0805_2012Metric -> A-PCENGINE:SMD_0805_Narrow
Changed lines of the file:
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@@
       (effects (font (size 1.27 1.27)) (justify left))
     )
-    (property "Footprint" "Capacitor_SMD:C_0805_2012Metric" (at 277.8252 144.78 0)
+    (property "Footprint" "A-PCENGINE:SMD_0805_Narrow" (at 277.8252 144.78 0)
       (effects (font (size 1.27 1.27)) hide)
     )
@@
       (effects (font (size 1.27 1.27)) (justify left))
     )
-    (property "Footprint" "Capacitor_SMD:C_0805_2012Metric" (at 206.7052 205.74 0)
+    (property "Footprint" "A-PCENGINE:SMD_0805_Narrow" (at 206.7052 205.74 0)
       (effects (font (size 1.27 1.27)) hide)
     )
@@
       (effects (font (size 1.27 1.27)) (justify left))
     )
-    (property "Footprint" "Capacitor_SMD:C_0805_2012Metric" (at 277.8252 85.09 0)
+    (property "Footprint" "A-PCENGINE:SMD_0805_Narrow" (at 277.8252 85.09 0)
       (effects (font (size 1.27 1.27)) hide)
     )
@@
       (effects (font (size 1.27 1.27)) (justify left))
     )
-    (property "Footprint" "Capacitor_SMD:C_0805_2012Metric" (at 232.1052 205.74 0)
+    (property "Footprint" "A-PCENGINE:SMD_0805_Narrow" (at 232.1052 205.74 0)
       (effects (font (size 1.27 1.27)) hide)
     )
@@
       (effects (font (size 1.27 1.27)) (justify left))
     )
-    (property "Footprint" "Capacitor_SMD:C_0805_2012Metric" (at 155.2448 140.97 0)
+    (property "Footprint" "A-PCENGINE:SMD_0805_Narrow" (at 155.2448 140.97 0)
       (effects (font (size 1.27 1.27)) hide)
     )
@@
       (effects (font (size 1.27 1.27)) (justify left))
     )
-    (property "Footprint" "Capacitor_SMD:C_0805_2012Metric" (at 219.4052 205.74 0)
-      (effects (font (size 1.27 1.27)) hide)
-    )
+    (property "Footprint" "A-PCENGINE:SMD_0805_Narrow" (at 219.4052 205.74 0)
+      (effects (font (size 1.27 1.27)) hide)
+    )

Commit message: Fix DRC errors.
Parts:
- added TP1: ~, A-PCENGINE:Test_Point_1.5mm_THT_NoSilk, symbol Connector:TestPoint
- renumbered IC9001 to IC904, IC9002 to IC905
Connections:
- net at IC902.27 (DISP): now also TP1.1
- no-connect marks 9 -> 8
Changed lines of the file:
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@@
   (no_connect (at 166.37 74.93))
   (no_connect (at 166.37 87.63))
-  (no_connect (at 201.93 163.83))
   (no_connect (at 166.37 80.01))
   (no_connect (at 166.37 85.09))
@@
     (stroke (width 0) (type default))
   )
+  (wire (pts (xy 201.93 163.83) (xy 206.502 163.83))
+    (stroke (width 0) (type default))
+  )
   (bus (pts (xy 237.49 114.3) (xy 237.49 111.76))
     (stroke (width 0) (type default))
@@
   )
   (wire (pts (xy 275.59 72.39) (xy 276.86 72.39))
+    (stroke (width 0) (type default))
+  )
+  (wire (pts (xy 206.502 163.83) (xy 206.502 167.64))
     (stroke (width 0) (type default))
   )
@@
   (symbol (lib_id "PC-Engine:M20256") (at 261.62 97.79 0) (unit 1)
     (in_bom yes) (on_board yes) (dnp no)
-    (property "Reference" "IC9002" (at 261.62 97.79 0)
+    (property "Reference" "IC905" (at 261.62 97.79 0)
       (effects (font (size 1.27 1.27)))
     )
@@
       (project "PCE"
         (path "/c1c718c6-a427-431e-a18b-e46f94ae8e09/ed9120da-14d8-40be-9026-fb246d72bf2f"
-          (reference "IC9002") (unit 1)
+          (reference "IC905") (unit 1)
         )
       )
@@
   (symbol (lib_id "PC-Engine:M20256") (at 261.62 38.1 0) (unit 1)
     (in_bom yes) (on_board yes) (dnp no)
-    (property "Reference" "IC9001" (at 261.62 38.1 0)
+    (property "Reference" "IC904" (at 261.62 38.1 0)
       (effects (font (size 1.27 1.27)))
     )
@@
       (project "PCE"
         (path "/c1c718c6-a427-431e-a18b-e46f94ae8e09/ed9120da-14d8-40be-9026-fb246d72bf2f"
-          (reference "IC9001") (unit 1)
+          (reference "IC904") (unit 1)
         )
       )
@@
         )
       )
+    )
+  )
+  (symbol (lib_id "Connector:TestPoint") (at 206.502 167.64 180) (unit 1)
+    (in_bom yes) (on_board yes) (dnp no)
+    (property "Reference" "TP1" (at 206.502 177.165 90)
+      (effects (font (size 1.27 1.27)) (justify right))
+    )
+    (property "Value" "~" (at 208.407 172.212 0)
+      (effects (font (size 1.27 1.27)) (justify right))
+    )
+    (property "Footprint" "A-PCENGINE:Test_Point_1.5mm_THT_NoSilk" (at 201.422 167.64 0)
+      (effects (font (size 1.27 1.27)) hide)
+    )
+    (property "Datasheet" "~" (at 201.422 167.64 0)
+      (effects (font (size 1.27 1.27)) hide)
+    )
+    (pin "1")
+    (instances
+      (project "PCE"
+        (path "/c1c718c6-a427-431e-a18b-e46f94ae8e09/bb2f9872-1813-43e0-bcfc-5c5426bf43ce"
+          (reference "TP1") (unit 1)
+        )
+        (path "/c1c718c6-a427-431e-a18b-e46f94ae8e09/ed9120da-14d8-40be-9026-fb246d72bf2f"
+          (reference "TP65") (unit 1)
+        )
+      )

Commit message: General clean-up.
Parts:
- removed TP1: ~, A-PCENGINE:Test_Point_1.5mm_THT_NoSilk, symbol Connector:TestPoint
- added TP101: ~, A-PCENGINE:Test_Point_2mm_THT, symbol Connector:TestPoint
Connections:
- net at IC902.27 (DISP): now also TP101.1
Changed lines of the file:
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@@
+    )
+  )
+  (symbol (lib_id "Connector:TestPoint") (at 206.502 167.64 180) (unit 1)
+    (in_bom yes) (on_board yes) (dnp no)
+    (property "Reference" "TP101" (at 206.502 177.165 90)
+      (effects (font (size 1.27 1.27)) (justify right))
+    )
+    (property "Value" "~" (at 208.407 172.212 0)
+      (effects (font (size 1.27 1.27)) (justify right))
+    )
+    (property "Footprint" "A-PCENGINE:Test_Point_2mm_THT" (at 201.422 167.64 0)
+      (effects (font (size 1.27 1.27)) hide)
+    )
+    (property "Datasheet" "~" (at 201.422 167.64 0)
+      (effects (font (size 1.27 1.27)) hide)
+    )
+    (pin "1")
+    (instances
+      (project "PCE"
+        (path "/c1c718c6-a427-431e-a18b-e46f94ae8e09/bb2f9872-1813-43e0-bcfc-5c5426bf43ce"
+          (reference "TP101") (unit 1)
+        )
+        (path "/c1c718c6-a427-431e-a18b-e46f94ae8e09/ed9120da-14d8-40be-9026-fb246d72bf2f"
+          (reference "TP1") (unit 1)
+        )
+      )
     )
   )
@@
         )
       )
-    )
-  )
-  (symbol (lib_id "Connector:TestPoint") (at 206.502 167.64 180) (unit 1)
-    (in_bom yes) (on_board yes) (dnp no)
-    (property "Reference" "TP1" (at 206.502 177.165 90)
-      (effects (font (size 1.27 1.27)) (justify right))
-    )
-    (property "Value" "~" (at 208.407 172.212 0)
-      (effects (font (size 1.27 1.27)) (justify right))
-    )
-    (property "Footprint" "A-PCENGINE:Test_Point_1.5mm_THT_NoSilk" (at 201.422 167.64 0)
-      (effects (font (size 1.27 1.27)) hide)
-    )
-    (property "Datasheet" "~" (at 201.422 167.64 0)
-      (effects (font (size 1.27 1.27)) hide)
-    )
-    (pin "1")
-    (instances
-      (project "PCE"
-        (path "/c1c718c6-a427-431e-a18b-e46f94ae8e09/bb2f9872-1813-43e0-bcfc-5c5426bf43ce"
-          (reference "TP1") (unit 1)
-        )
-        (path "/c1c718c6-a427-431e-a18b-e46f94ae8e09/ed9120da-14d8-40be-9026-fb246d72bf2f"
-          (reference "TP65") (unit 1)
-        )
-      )
