File: vdc.kicad_sch (KiCad schematic)
At the start: 10 parts, among them IC902 HUC6270, IC904 M20256, IC905 M20256

Commit message: Add known capacitor values to schematic. PCB changes: - Corrected C332 -> C322 - Corrected C929 -> C962 - Added missing C166 (extra decoupling for IC105)
Parts:
- C102, C104, C106, C904, C914: value 0.1uF -> 100nF
Changed lines of the file:
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@@
       (effects (font (size 1.27 1.27)) (justify left))
     )
-    (property "Value" "0.1uF" (at 278.13 144.78 0)
+    (property "Value" "100nF" (at 278.13 144.78 0)
       (effects (font (size 1.27 1.27)) (justify left))
     )
@@
       (effects (font (size 1.27 1.27)) (justify left))
     )
-    (property "Value" "0.1uF" (at 209.55 203.2 0)
+    (property "Value" "100nF" (at 209.55 203.2 0)
       (effects (font (size 1.27 1.27)) (justify left))
     )
@@
       (effects (font (size 1.27 1.27)) (justify left))
     )
-    (property "Value" "0.1uF" (at 278.13 85.09 0)
+    (property "Value" "100nF" (at 278.13 85.09 0)
       (effects (font (size 1.27 1.27)) (justify left))
     )
@@
       (effects (font (size 1.27 1.27)) (justify left))
     )
-    (property "Value" "0.1uF" (at 234.95 203.2 0)
+    (property "Value" "100nF" (at 234.95 203.2 0)
       (effects (font (size 1.27 1.27)) (justify left))
     )
@@
       (effects (font (size 1.27 1.27)) (justify left))
     )
-    (property "Value" "0.1uF" (at 152.4 139.065 0)
+    (property "Value" "100nF" (at 152.4 139.065 0)
       (effects (font (size 1.27 1.27)) (justify left))
     )
@@
       (effects (font (size 1.27 1.27)) (justify left))
     )
-    (property "Value" "0.1uF" (at 222.25 203.2 0)
-      (effects (font (size 1.27 1.27)) (justify left))
-    )
+    (property "Value" "100nF" (at 222.25 203.2 0)
+      (effects (font (size 1.27 1.27)) (justify left))
+    )

Commit message: More schematic clean-up/annotation.
Other:
- company: (none) -> By Cosam
- title: PC Engine Video Display Controller and VRAM -> PC Engine Duo Video Display Controller and VRAM
Changed lines of the file:
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@@
   (paper "A3")
   (title_block
-    (title "PC Engine Video Display Controller and VRAM")
-    (date "2023-11-01")
-    (rev "1.0")
-    (comment 1 "Reverse engineered from original PWA-3285-A board by Cosam")
-    (comment 3 "WORK IN PROGRESS")
+    (title "PC Engine Duo Video Display Controller and VRAM")
+    (date "2023-11-03")
+    (rev "1.1")
+    (company "By Cosam")
+    (comment 1 "https://github.com/Board-Folk/PC-Engine-Duo")
+    (comment 2 "For contributions or corrections please visit:")
+    (comment 3 "Additional parts reverse engineered from original PWA-3285-A board.")
+    (comment 4 "Parts common to PC Engine adapted from TurboGrafx-16 schematics.")
   )
   (junction (at 218.44 195.58) (diameter 0) (color 0 0 0 0)
