File: cpu.kicad_sch (KiCad schematic)
At the start: 32 parts, among them IC901 HUC6280, IC906 LC3664BML-10

Commit message: Bunch of passives and what-not.
Parts:
- C951, R901: footprint A-PCENGINE:SMD_0805_Narrow -> A-PCENGINE:SMD_0805_Narrow_Long
- D901: footprint A-PCENGINE:Diode_SMD -> A-PCENGINE:Transistor_SMD; symbol Device:D -> PC-Engine:D-1-3
- Rx999: renamed from R921; footprint A-PCENGINE:SMD_0805_Narrow -> A-PCENGINE:SMD_0805_Narrow_Long
- renumbered C123 to Cx123, R102 to R903, R103 to R904, R105 to R905, Rx114 to R906
Connections:
- net XB is gone; now on net GND: IC901.30 (K7)
- net +5V: now also D901.3 (K); no longer D901.1 (K)
- net ~{RST-OSC}: now also D901.1 (A); no longer D901.2 (A)
Changed lines of the file:
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@@
   (junction (at 170.18 254) (diameter 0) (color 0 0 0 0)
+  )
+  (junction (at 180.34 181.61) (diameter 0) (color 0 0 0 0)
   )
   (junction (at 132.08 241.3) (diameter 0) (color 0 0 0 0)
@@
     (stroke (width 0) (type default))
   )
-  (wire (pts (xy 187.96 138.43) (xy 193.04 138.43))
+  (wire (pts (xy 173.355 138.43) (xy 193.04 138.43))
     (stroke (width 0) (type default))
   )
@@
     (stroke (width 0) (type default))
   )
+  (wire (pts (xy 173.355 138.43) (xy 173.355 181.61))
+    (stroke (width 0) (type default))
+  )
   (wire (pts (xy 231.14 163.83) (xy 231.14 220.98))
     (stroke (width 0) (type default))
@@
   )
   (wire (pts (xy 128.27 207.01) (xy 128.27 203.2))
+    (stroke (width 0) (type default))
+  )
+  (wire (pts (xy 173.355 181.61) (xy 180.34 181.61))
     (stroke (width 0) (type default))
   )
@@
     )
   )
-  (global_label "XB" (shape output) (at 187.96 138.43 180) (fields_autoplaced)
-    (effects (font (size 1.27 1.27)) (justify right))
-    (property "Intersheetrefs" "${INTERSHEET_REFS}" (at 182.5747 138.43 0)
-      (effects (font (size 1.27 1.27)) (justify right) hide)
-    )
-  )
   (global_label "RDY" (shape output) (at 52.07 39.37 180) (fields_autoplaced)
     (effects (font (size 1.27 1.27)) (justify right))
@@
       (effects (font (size 1.27 1.27)) (justify left))
     )
-    (property "Footprint" "A-PCENGINE:SMD_0805_Narrow" (at 156.972 46.99 90)
+    (property "Footprint" "A-PCENGINE:SMD_0805_Narrow_Long" (at 156.972 46.99 90)
       (effects (font (size 1.27 1.27)) hide)
     )
@@
   (symbol (lib_id "Device:R") (at 135.89 67.31 0) (unit 1)
     (in_bom yes) (on_board yes) (dnp no) (fields_autoplaced)
-    (property "Reference" "Rx114" (at 138.43 66.04 0)
+    (property "Reference" "R906" (at 138.43 66.04 0)
       (effects (font (size 1.27 1.27)) (justify left))
     )
@@
       (project "PCE"
         (path "/c1c718c6-a427-431e-a18b-e46f94ae8e09/1d91d06a-381a-4a70-bfc1-2abf4d159a91"
-          (reference "Rx114") (unit 1)
+          (reference "R906") (unit 1)
         )
       )
@@
   (symbol (lib_id "Device:R") (at 167.64 58.42 0) (unit 1)
     (in_bom yes) (on_board yes) (dnp no) (fields_autoplaced)
-    (property "Reference" "R103" (at 170.18 57.785 0)
-      (effects (font (size 1.27 1.27)) (justify left))
-    )
-    (property "Value" "4.7K" (at 170.18 60.325 0)
+    (property "Reference" "R904" (at 170.18 57.15 0)
+      (effects (font (size 1.27 1.27)) (justify left))
+    )
+    (property "Value" "4.7K" (at 170.18 59.69 0)
       (effects (font (size 1.27 1.27)) (justify left))
     )
@@
       (project "PCE"
         (path "/c1c718c6-a427-431e-a18b-e46f94ae8e09/1d91d06a-381a-4a70-bfc1-2abf4d159a91"
-          (reference "R103") (unit 1)
+          (reference "R904") (unit 1)
         )
       )
@@
   (symbol (lib_id "Device:R") (at 127 58.42 180) (unit 1)
     (in_bom yes) (on_board yes) (dnp no) (fields_autoplaced)
-    (property "Reference" "R105" (at 129.54 57.785 0)
+    (property "Reference" "R905" (at 129.54 57.15 0)
       (effects (font (size 1.27 1.27)) (justify right))
     )
-    (property "Value" "4.7K" (at 129.54 60.325 0)
+    (property "Value" "4.7K" (at 129.54 59.69 0)
       (effects (font (size 1.27 1.27)) (justify right))
     )
@@
       (project "PCE"
         (path "/c1c718c6-a427-431e-a18b-e46f94ae8e09/1d91d06a-381a-4a70-bfc1-2abf4d159a91"
-          (reference "R105") (unit 1)
+          (reference "R905") (unit 1)
         )
       )
@@
   (symbol (lib_id "Device:C") (at 180.34 171.45 0) (unit 1)
     (in_bom yes) (on_board yes) (dnp no)
-    (property "Reference" "C123" (at 184.15 170.815 0)
+    (property "Reference" "Cx123" (at 184.15 170.815 0)
       (effects (font (size 1.27 1.27)) (justify left))
     )
@@
       (project "PCE"
         (path "/c1c718c6-a427-431e-a18b-e46f94ae8e09/1d91d06a-381a-4a70-bfc1-2abf4d159a91"
-          (reference "C123") (unit 1)
+          (reference "Cx123") (unit 1)
         )
       )
@@
   (symbol (lib_id "Device:R") (at 144.78 76.2 0) (unit 1)
     (in_bom yes) (on_board yes) (dnp no) (fields_autoplaced)
-    (property "Reference" "R102" (at 147.32 75.565 0)
-      (effects (font (size 1.27 1.27)) (justify left))
-    )
-    (property "Value" "4.7K" (at 147.32 78.105 0)
+    (property "Reference" "R903" (at 147.32 74.93 0)
+      (effects (font (size 1.27 1.27)) (justify left))
+    )
+    (property "Value" "4.7K" (at 147.32 77.47 0)
       (effects (font (size 1.27 1.27)) (justify left))
     )
@@
       (project "PCE"
         (path "/c1c718c6-a427-431e-a18b-e46f94ae8e09/1d91d06a-381a-4a70-bfc1-2abf4d159a91"
-          (reference "R102") (unit 1)
+          (reference "R903") (unit 1)
         )
       )
@@
     )
   )
-  (symbol (lib_id "Device:D") (at 149.86 58.42 270) (unit 1)
+  (symbol (lib_id "PC-Engine:D-1-3") (at 149.86 58.42 270) (unit 1)
     (in_bom yes) (on_board yes) (dnp no) (fields_autoplaced)
     (property "Reference" "D901" (at 152.4 57.15 90)
@@
       (effects (font (size 1.27 1.27)) (justify left))
     )
-    (property "Footprint" "A-PCENGINE:Diode_SMD" (at 149.86 58.42 0)
+    (property "Footprint" "A-PCENGINE:Transistor_SMD" (at 149.86 58.42 0)
       (effects (font (size 1.27 1.27)) hide)
     )
@@
       (effects (font (size 1.27 1.27)) hide)
     )
-    (property "Sim.Pins" "1=K 2=A" (at 149.86 58.42 0)
-      (effects (font (size 1.27 1.27)) hide)
-    )
-    (pin "1")
-    (pin "2")
+    (property "Sim.Pins" "1=A 3=K" (at 147.955 58.42 0)
+      (effects (font (size 1.27 1.27)) hide)
+    )
+    (pin "1")
+    (pin "2")
+    (pin "3")
     (instances
       (project "PCE"
@@
       (effects (font (size 1.27 1.27)) (justify left))
     )
-    (property "Footprint" "A-PCENGINE:SMD_0805_Narrow" (at 112.7252 113.03 0)
+    (property "Footprint" "A-PCENGINE:SMD_0805_Narrow_Long" (at 112.7252 113.03 0)
       (effects (font (size 1.27 1.27)) hide)
     )
@@
   (symbol (lib_id "Device:R") (at 115.57 180.34 0) (unit 1)
     (in_bom yes) (on_board yes) (dnp no) (fields_autoplaced)
-    (property "Reference" "R921" (at 118.11 179.07 0)
+    (property "Reference" "Rx999" (at 118.11 179.07 0)
       (effects (font (size 1.27 1.27)) (justify left))
     )
@@
       (effects (font (size 1.27 1.27)) (justify left))
     )
-    (property "Footprint" "A-PCENGINE:SMD_0805_Narrow" (at 113.792 180.34 90)
+    (property "Footprint" "A-PCENGINE:SMD_0805_Narrow_Long" (at 113.792 180.34 90)
       (effects (font (size 1.27 1.27)) hide)
     )
@@
       (project "PCE"
         (path "/c1c718c6-a427-431e-a18b-e46f94ae8e09/1d91d06a-381a-4a70-bfc1-2abf4d159a91"
-          (reference "R921") (unit 1)
-        )
-      )
+          (reference "Rx999") (unit 1)
+        )
+      )

Commit message: More passives, custom footprints, etc.
Parts:
- removed C105: 10uF 16V, A-PCENGINE:Elec_P5.00mm, symbol Device:C_Polarized
- removed ICX108: μPC358C, Package_SO:HSOP-32-1EP_7.5x11mm_P0.65mm_EP4.7x4.7mm, symbol Amplifier_Operational:LM358
- C906: footprint A-PCENGINE:SMD_0805_Narrow -> A-PCENGINE:SMD_0805_Narrow_Long; now in the parts list
- C944, R907, R908, R909: footprint A-PCENGINE:SMD_0805_Narrow -> A-PCENGINE:SMD_0805_Narrow_Long
- IC906: footprint Package_SO:SOIC-28W_7.5x17.9mm_P1.27mm -> A-PCENGINE:HSRM20256LM
Changed lines of the file:
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@@
-    (stroke (width 0) (type default))
-  )
-  (wire (pts (xy 213.36 255.27) (xy 213.36 256.54))
     (stroke (width 0) (type default))
   )
@@
   )
   (wire (pts (xy 95.25 123.19) (xy 95.25 143.51))
-    (stroke (width 0) (type default))
-  )
-  (wire (pts (xy 213.36 238.76) (xy 213.36 240.03))
     (stroke (width 0) (type default))
   )
@@
         (path "/c1c718c6-a427-431e-a18b-e46f94ae8e09/1d91d06a-381a-4a70-bfc1-2abf4d159a91"
           (reference "C901") (unit 1)
+        )
+      )
+    )
+  )
+  (symbol (lib_id "Device:C") (at 322.58 101.6 0) (unit 1)
+    (in_bom yes) (on_board yes) (dnp no) (fields_autoplaced)
+    (property "Reference" "C906" (at 326.39 100.33 0)
+      (effects (font (size 1.27 1.27)) (justify left))
+    )
+    (property "Value" "0.1uF" (at 326.39 102.87 0)
+      (effects (font (size 1.27 1.27)) (justify left))
+    )
+    (property "Footprint" "A-PCENGINE:SMD_0805_Narrow_Long" (at 323.5452 105.41 0)
+      (effects (font (size 1.27 1.27)) hide)
+    )
+    (property "Datasheet" "~" (at 322.58 101.6 0)
+      (effects (font (size 1.27 1.27)) hide)
+    )
+    (pin "1")
+    (pin "2")
+    (instances
+      (project "PCE"
+        (path "/c1c718c6-a427-431e-a18b-e46f94ae8e09/1d91d06a-381a-4a70-bfc1-2abf4d159a91"
+          (reference "C906") (unit 1)
         )
       )
@@
     )
   )
-  (symbol (lib_id "power:+5V") (at 213.36 238.76 0) (unit 1)
-    (in_bom yes) (on_board yes) (dnp no) (fields_autoplaced)
-    (property "Reference" "#PWR054" (at 213.36 242.57 0)
-      (effects (font (size 1.27 1.27)) hide)
-    )
-    (property "Value" "+5V" (at 213.36 234.95 0)
-      (effects (font (size 1.27 1.27)))
-    )
-    (property "Footprint" "" (at 213.36 238.76 0)
-      (effects (font (size 1.27 1.27)) hide)
-    )
-    (property "Datasheet" "" (at 213.36 238.76 0)
-      (effects (font (size 1.27 1.27)) hide)
-    )
-    (pin "1")
-    (instances
-      (project "PCE"
-        (path "/c1c718c6-a427-431e-a18b-e46f94ae8e09/1d91d06a-381a-4a70-bfc1-2abf4d159a91"
-          (reference "#PWR054") (unit 1)
-        )
-      )
-    )
-  )
   (symbol (lib_id "power:+5V") (at 180.34 158.75 0) (unit 1)
     (in_bom yes) (on_board yes) (dnp no) (fields_autoplaced)
@@
     )
   )
-  (symbol (lib_id "Device:C_Polarized") (at 128.27 199.39 0) (unit 1)
-    (in_bom yes) (on_board yes) (dnp no) (fields_autoplaced)
-    (property "Reference" "C105" (at 132.08 197.866 0)
-      (effects (font (size 1.27 1.27)) (justify left))
-    )
-    (property "Value" "10uF 16V" (at 132.08 200.406 0)
-      (effects (font (size 1.27 1.27)) (justify left))
-    )
-    (property "Footprint" "A-PCENGINE:Elec_P5.00mm" (at 129.2352 203.2 0)
-      (effects (font (size 1.27 1.27)) hide)
-    )
-    (property "Datasheet" "~" (at 128.27 199.39 0)
-      (effects (font (size 1.27 1.27)) hide)
-    )
-    (pin "1")
-    (pin "2")
-    (instances
-      (project "PCE"
-        (path "/c1c718c6-a427-431e-a18b-e46f94ae8e09/1d91d06a-381a-4a70-bfc1-2abf4d159a91"
-          (reference "C105") (unit 1)
-        )
-      )
-    )
-  )
   (symbol (lib_id "power:+5VA") (at 115.57 168.91 0) (unit 1)
     (in_bom yes) (on_board yes) (dnp no) (fields_autoplaced)
@@
         (path "/c1c718c6-a427-431e-a18b-e46f94ae8e09/1d91d06a-381a-4a70-bfc1-2abf4d159a91"
           (reference "R903") (unit 1)
-        )
-      )
-    )
-  )
-  (symbol (lib_id "Amplifier_Operational:LM358") (at 215.9 247.65 0) (unit 3)
-    (in_bom yes) (on_board yes) (dnp no)
-    (property "Reference" "ICX108" (at 220.98 246.38 0)
-      (effects (font (size 1.27 1.27)))
-    )
-    (property "Value" "μPC358C" (at 220.98 248.92 0)
-      (effects (font (size 1.27 1.27)))
-    )
-    (property "Footprint" "Package_SO:HSOP-32-1EP_7.5x11mm_P0.65mm_EP4.7x4.7mm" (at 215.9 247.65 0)
-      (effects (font (size 1.27 1.27)) hide)
-    )
-    (property "Datasheet" "http://www.ti.com/lit/ds/symlink/lm2904-n.pdf" (at 215.9 247.65 0)
-      (effects (font (size 1.27 1.27)) hide)
-    )
-    (pin "1")
-    (pin "2")
-    (pin "3")
-    (pin "5")
-    (pin "6")
-    (pin "7")
-    (pin "4")
-    (pin "8")
-    (instances
-      (project "PCE"
-        (path "/c1c718c6-a427-431e-a18b-e46f94ae8e09/1d91d06a-381a-4a70-bfc1-2abf4d159a91"
-          (reference "ICX108") (unit 3)
-        )
-      )
-    )
-  )
-  (symbol (lib_id "power:GND") (at 213.36 256.54 0) (unit 1)
-    (in_bom yes) (on_board yes) (dnp no) (fields_autoplaced)
-    (property "Reference" "#PWR051" (at 213.36 262.89 0)
-      (effects (font (size 1.27 1.27)) hide)
-    )
-    (property "Value" "GND" (at 213.36 261.62 0)
-      (effects (font (size 1.27 1.27)))
-    )
-    (property "Footprint" "" (at 213.36 256.54 0)
-      (effects (font (size 1.27 1.27)) hide)
-    )
-    (property "Datasheet" "" (at 213.36 256.54 0)
-      (effects (font (size 1.27 1.27)) hide)
-    )
-    (pin "1")
-    (instances
-      (project "PCE"
-        (path "/c1c718c6-a427-431e-a18b-e46f94ae8e09/1d91d06a-381a-4a70-bfc1-2abf4d159a91"
-          (reference "#PWR051") (unit 1)
         )
       )
@@
       (effects (font (size 1.27 1.27)) (justify left))
     )
-    (property "Footprint" "A-PCENGINE:SMD_0805_Narrow" (at 71.882 62.23 90)
+    (property "Footprint" "A-PCENGINE:SMD_0805_Narrow_Long" (at 71.882 62.23 90)
       (effects (font (size 1.27 1.27)) hide)
     )
@@
         (path "/c1c718c6-a427-431e-a18b-e46f94ae8e09/1d91d06a-381a-4a70-bfc1-2abf4d159a91"
           (reference "R908") (unit 1)
-        )
-      )
-    )
-  )
-  (symbol (lib_id "Amplifier_Operational:LM358") (at 148.59 191.77 0) (unit 2)
-    (in_bom yes) (on_board yes) (dnp no) (fields_autoplaced)
-    (property "Reference" "ICX108" (at 148.59 182.88 0)
-      (effects (font (size 1.27 1.27)))
-    )
-    (property "Value" "μPC358C" (at 148.59 185.42 0)
-      (effects (font (size 1.27 1.27)))
-    )
-    (property "Footprint" "A-PCENGINE:DIP-8" (at 148.59 191.77 0)
-      (effects (font (size 1.27 1.27)) hide)
-    )
-    (property "Datasheet" "http://www.ti.com/lit/ds/symlink/lm2904-n.pdf" (at 148.59 191.77 0)
-      (effects (font (size 1.27 1.27)) hide)
-    )
-    (pin "1")
-    (pin "2")
-    (pin "3")
-    (pin "5")
-    (pin "6")
-    (pin "7")
-    (pin "4")
-    (pin "8")
-    (instances
-      (project "PCE"
-        (path "/c1c718c6-a427-431e-a18b-e46f94ae8e09/1d91d06a-381a-4a70-bfc1-2abf4d159a91"
-          (reference "ICX108") (unit 2)
         )
       )
@@
       (effects (font (size 1.27 1.27)))
     )
-    (property "Footprint" "A-PCENGINE:SMD_0805_Narrow" (at 81.28 56.388 90)
+    (property "Footprint" "A-PCENGINE:SMD_0805_Narrow_Long" (at 81.28 56.388 90)
       (effects (font (size 1.27 1.27)) hide)
     )
@@
       (effects (font (size 1.27 1.27)) (justify left))
     )
-    (property "Footprint" "A-PCENGINE:SMD_0805_Narrow" (at 56.642 62.23 90)
+    (property "Footprint" "A-PCENGINE:SMD_0805_Narrow_Long" (at 56.642 62.23 90)
       (effects (font (size 1.27 1.27)) hide)
     )
@@
       (effects (font (size 1.27 1.27)))
     )
-    (property "Footprint" "A-PCENGINE:SMD_0805_Narrow" (at 69.85 53.6448 0)
+    (property "Footprint" "A-PCENGINE:SMD_0805_Narrow_Long" (at 69.85 53.6448 0)
       (effects (font (size 1.27 1.27)) hide)
     )
@@
       (effects (font (size 1.27 1.27)))
     )
-    (property "Footprint" "Package_SO:SOIC-28W_7.5x17.9mm_P1.27mm" (at 303.53 58.42 0)
+    (property "Footprint" "A-PCENGINE:HSRM20256LM" (at 303.53 58.42 0)
       (effects (font (size 1.27 1.27)) hide)
     )
@@
         )
       )
-    )
-  )
-  (symbol (lib_id "Device:C") (at 322.58 101.6 0) (unit 1)
-    (in_bom no) (on_board no) (dnp no)
-    (property "Reference" "C906" (at 326.39 100.965 0)
-      (effects (font (size 1.27 1.27)) (justify left))
-    )
-    (property "Value" "0.1uF" (at 326.39 103.505 0)
-      (effects (font (size 1.27 1.27)) (justify left))
-    )
-    (property "Footprint" "A-PCENGINE:SMD_0805_Narrow" (at 323.5452 105.41 0)
-      (effects (font (size 1.27 1.27)) hide)
-    )
-    (property "Datasheet" "~" (at 322.58 101.6 0)
-      (effects (font (size 1.27 1.27)) hide)
-    )
-    (property "Sim.Enable" "0" (at 322.58 101.6 0)
-      (effects (font (size 1.27 1.27)) hide)
-    )
-    (pin "1")
-    (pin "2")
-    (instances
-      (project "PCE"
-        (path "/c1c718c6-a427-431e-a18b-e46f94ae8e09/1d91d06a-381a-4a70-bfc1-2abf4d159a91"
-          (reference "C906") (unit 1)
-        )
-      )

Commit message: Top layer first draft.
Parts:
- renumbered R152 to Rx152
Changed lines of the file:
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@@
   (symbol (lib_id "Device:R") (at 115.57 199.39 0) (unit 1)
     (in_bom yes) (on_board yes) (dnp no) (fields_autoplaced)
-    (property "Reference" "R152" (at 118.11 198.755 0)
+    (property "Reference" "Rx152" (at 118.11 198.12 0)
       (effects (font (size 1.27 1.27)) (justify left))
     )
-    (property "Value" "4.7K" (at 118.11 201.295 0)
+    (property "Value" "4.7K" (at 118.11 200.66 0)
       (effects (font (size 1.27 1.27)) (justify left))
     )
@@
       (project "PCE"
         (path "/c1c718c6-a427-431e-a18b-e46f94ae8e09/1d91d06a-381a-4a70-bfc1-2abf4d159a91"
-          (reference "R152") (unit 1)
+          (reference "Rx152") (unit 1)
         )
       )

Commit message: More passives on back.
Parts:
- removed Cx123: 0.1uf, A-PCENGINE:SMD_0805_Narrow, symbol Device:C
- added C952: ~, A-PCENGINE:CP_2010_XL, symbol Device:C_Polarized
- added C965: ~, A-PCENGINE:SMD_0805_Narrow, symbol Device:C
- added Q901: L6, A-PCENGINE:Transistor_SMD, symbol Device:Q_NPN_CBE
- added R912, R931: ~, A-PCENGINE:SMD_0805_Narrow_Long, symbol Device:R
- added TP1: ~, A-PCENGINE:Test_Point_1.5mm, symbol Connector:TestPoint
- R910: renamed from Rx152; value 4.7K -> ~; footprint A-PCENGINE:SMD_0805_Narrow -> A-PCENGINE:SMD_0805_Narrow_Long
- R911: renamed from Rx999; value 4.7K -> ~; footprint A-PCENGINE:SMD_0805_Narrow_Long -> A-PCENGINE:SMD_0805_Narrow
Connections:
- net +5VA: now also Q901.1 (C)
- net AGND: now also C952.1, Q901.3 (E), R912.1, R931.1, TP1.1
- net GNDA: now also C952.2, C965.2, R912.2, R931.2
- net at R910.1, R911.2: now also C965.1, Q901.2 (B)
Other:
- moved on the sheet: R911

Commit message: Fix DRC errors.
Parts:
- added TP1: ~, A-PCENGINE:Test_Point_1.5mm_THT_NoSilk, symbol Connector:TestPoint
Connections:
- net ~{WR}: now also TP1.1
- net LOUT renamed AUDIO-L
- net ROUT renamed AUDIO-R
Changed lines of the file:
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@@
   (junction (at 160.02 191.77) (diameter 0) (color 0 0 0 0)
+  )
+  (junction (at 241.3 123.19) (diameter 0) (color 0 0 0 0)
   )
   (junction (at 190.5 176.53) (diameter 0) (color 0 0 0 0)
@@
     (stroke (width 0) (type default))
   )
+  (wire (pts (xy 241.3 121.412) (xy 241.3 123.19))
+    (stroke (width 0) (type default))
+  )
   (wire (pts (xy 233.68 166.37) (xy 233.68 226.06))
     (stroke (width 0) (type default))
@@
     (stroke (width 0) (type default))
   )
+  (wire (pts (xy 241.3 123.19) (xy 269.24 123.19))
+    (stroke (width 0) (type default))
+  )
   (wire (pts (xy 135.89 27.94) (xy 144.78 27.94))
     (stroke (width 0) (type default))
@@
     (stroke (width 0) (type default))
   )
-  (wire (pts (xy 228.6 123.19) (xy 269.24 123.19))
+  (wire (pts (xy 228.6 123.19) (xy 241.3 123.19))
     (stroke (width 0) (type default))
   )
@@
     (stroke (width 0) (type default))
   )
-  (wire (pts (xy 228.6 157.48) (xy 308.61 157.48))
+  (wire (pts (xy 228.6 157.48) (xy 306.07 157.48))
     (stroke (width 0) (type default))
   )
@@
     )
   )
-  (global_label "ROUT" (shape output) (at 308.61 157.48 0) (fields_autoplaced)
+  (global_label "AUDIO-R" (shape output) (at 306.07 157.48 0) (fields_autoplaced)
     (effects (font (size 1.27 1.27)) (justify left))
-    (property "Intersheetrefs" "${INTERSHEET_REFS}" (at 316.4144 157.48 0)
+    (property "Intersheetrefs" "${INTERSHEET_REFS}" (at 317.522 157.48 0)
       (effects (font (size 1.27 1.27)) (justify left) hide)
     )
@@
     )
   )
-  (global_label "LOUT" (shape output) (at 317.5 154.94 0) (fields_autoplaced)
+  (global_label "AUDIO-L" (shape output) (at 317.5 154.94 0) (fields_autoplaced)
     (effects (font (size 1.27 1.27)) (justify left))
-    (property "Intersheetrefs" "${INTERSHEET_REFS}" (at 325.0625 154.94 0)
+    (property "Intersheetrefs" "${INTERSHEET_REFS}" (at 328.7101 154.94 0)
       (effects (font (size 1.27 1.27)) (justify left) hide)
     )
@@
         )
       )
+    )
+  )
+  (symbol (lib_id "Connector:TestPoint") (at 241.3 121.412 0) (unit 1)
+    (in_bom yes) (on_board yes) (dnp no)
+    (property "Reference" "TP1" (at 241.3 111.887 90)
+      (effects (font (size 1.27 1.27)) (justify right))
+    )
+    (property "Value" "~" (at 239.395 116.84 0)
+      (effects (font (size 1.27 1.27)) (justify right))
+    )
+    (property "Footprint" "A-PCENGINE:Test_Point_1.5mm_THT_NoSilk" (at 246.38 121.412 0)
+      (effects (font (size 1.27 1.27)) hide)
+    )
+    (property "Datasheet" "~" (at 246.38 121.412 0)
+      (effects (font (size 1.27 1.27)) hide)
+    )
+    (pin "1")
+    (instances
+      (project "PCE"
+        (path "/c1c718c6-a427-431e-a18b-e46f94ae8e09/bb2f9872-1813-43e0-bcfc-5c5426bf43ce"
+          (reference "TP1") (unit 1)
+        )
+        (path "/c1c718c6-a427-431e-a18b-e46f94ae8e09/ed9120da-14d8-40be-9026-fb246d72bf2f"
+          (reference "TP65") (unit 1)
+        )
+        (path "/c1c718c6-a427-431e-a18b-e46f94ae8e09/1d91d06a-381a-4a70-bfc1-2abf4d159a91"
+          (reference "TP66") (unit 1)
+        )
+      )

Commit message: Add resistor values to schematics.
Parts:
- R901: value 33K -> 330K
- R905: value 4.7K -> 10K
- R910: value ~ -> 6.8K
- R911: value ~ -> 3.3K
- R912: value ~ -> 10K
- R931: value ~ -> 510
Changed lines of the file:
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@@
       (effects (font (size 1.27 1.27)) (justify left))
     )
-    (property "Value" "~" (at 118.11 200.66 0)
+    (property "Value" "6.8K" (at 118.11 200.66 0)
       (effects (font (size 1.27 1.27)) (justify left))
     )
@@
       (effects (font (size 1.27 1.27)) (justify left))
     )
-    (property "Value" "33K" (at 161.29 48.26 0)
+    (property "Value" "330K" (at 161.29 48.26 0)
       (effects (font (size 1.27 1.27)) (justify left))
     )
@@
       (effects (font (size 1.27 1.27)) (justify left))
     )
-    (property "Value" "~" (at 153.035 200.66 0)
+    (property "Value" "10K" (at 153.035 200.66 0)
       (effects (font (size 1.27 1.27)) (justify left))
     )
@@
       (effects (font (size 1.27 1.27)) (justify left))
     )
-    (property "Value" "~" (at 142.875 200.66 0)
+    (property "Value" "510" (at 142.875 200.66 0)
       (effects (font (size 1.27 1.27)) (justify left))
     )
@@
       (effects (font (size 1.27 1.27)) (justify right))
     )
-    (property "Value" "4.7K" (at 129.54 59.69 0)
+    (property "Value" "10K" (at 129.54 59.69 0)
       (effects (font (size 1.27 1.27)) (justify right))
     )
@@
       (effects (font (size 1.27 1.27)) (justify left))
     )
-    (property "Value" "~" (at 118.11 182.88 0)
-      (effects (font (size 1.27 1.27)) (justify left))
-    )
+    (property "Value" "3.3K" (at 118.11 182.88 0)
+      (effects (font (size 1.27 1.27)) (justify left))
+    )
