File: video.kicad_sch (KiCad schematic)
At the start: 35 parts, among them IC903 HUC6260, Q902 25C945, Q903 25A733, Q904 25C945

Commit message: Add known capacitor values to schematic. PCB changes: - Corrected C332 -> C322 - Corrected C929 -> C962 - Added missing C166 (extra decoupling for IC105)
Parts:
- C101: symbol Device:C_Polarized -> Device:C
- C104, C105, C106: value 0.1uF -> 100nF
- C107: value 220pF -> 200pF
Changed lines of the file:
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@@
       (effects (font (size 1.27 1.27)) (justify left))
     )
-    (property "Value" "0.1uF" (at 182.88 229.87 0)
+    (property "Value" "100nF" (at 182.88 229.87 0)
       (effects (font (size 1.27 1.27)) (justify left))
     )
@@
     )
   )
-  (symbol (lib_id "Device:C_Polarized") (at 106.68 92.71 270) (unit 1)
+  (symbol (lib_id "Device:C") (at 106.68 92.71 270) (unit 1)
     (in_bom yes) (on_board yes) (dnp no)
     (property "Reference" "C101" (at 106.68 88.9 90)
@@
       (effects (font (size 1.27 1.27)) (justify left))
     )
-    (property "Value" "0.1uF" (at 195.58 229.87 0)
+    (property "Value" "100nF" (at 195.58 229.87 0)
       (effects (font (size 1.27 1.27)) (justify left))
     )
@@
     )
   )
-  (symbol (lib_id "Device:C_Polarized") (at 106.68 127 270) (unit 1)
+  (symbol (lib_id "Device:C") (at 106.68 127 270) (unit 1)
     (in_bom yes) (on_board yes) (dnp no)
     (property "Reference" "C101" (at 106.68 123.19 90)
@@
     )
   )
-  (symbol (lib_id "Device:C_Polarized") (at 95.25 109.22 270) (unit 1)
+  (symbol (lib_id "Device:C") (at 95.25 109.22 270) (unit 1)
     (in_bom yes) (on_board yes) (dnp no)
     (property "Reference" "C101" (at 95.25 105.41 90)
@@
       (effects (font (size 1.27 1.27)) (justify left))
     )
-    (property "Value" "0.1uF" (at 170.18 229.87 0)
+    (property "Value" "100nF" (at 170.18 229.87 0)
       (effects (font (size 1.27 1.27)) (justify left))
     )
@@
       (effects (font (size 1.27 1.27)))
     )
-    (property "Value" "220pF" (at 106.68 157.48 90)
+    (property "Value" "200pF" (at 106.68 157.48 90)
       (effects (font (size 1.27 1.27)))
     )
@@
     )
   )
-  (symbol (lib_id "Device:C_Polarized") (at 95.25 132.08 270) (unit 1)
+  (symbol (lib_id "Device:C") (at 95.25 132.08 270) (unit 1)
     (in_bom yes) (on_board yes) (dnp no)
     (property "Reference" "C101" (at 95.25 128.27 90)
@@
     )
   )
-  (symbol (lib_id "Device:C_Polarized") (at 106.68 104.14 270) (unit 1)
+  (symbol (lib_id "Device:C") (at 106.68 104.14 270) (unit 1)
     (in_bom yes) (on_board yes) (dnp no)
     (property "Reference" "C101" (at 106.68 100.33 90)
@@
       (effects (font (size 1.27 1.27)) (justify left))
     )
-    (property "Value" "0.1uF" (at 153.67 229.87 0)
+    (property "Value" "100nF" (at 153.67 229.87 0)
       (effects (font (size 1.27 1.27)) (justify left))
     )
@@
     )
   )
-  (symbol (lib_id "Device:C_Polarized") (at 106.68 115.57 270) (unit 1)
+  (symbol (lib_id "Device:C") (at 106.68 115.57 270) (unit 1)
     (in_bom yes) (on_board yes) (dnp no)
     (property "Reference" "C101" (at 106.68 111.76 90)
@@
         )
         (path "/c1c718c6-a427-431e-a18b-e46f94ae8e09/c78d7e8a-3e65-46f4-91f4-96eb31925bea"
-          (reference "C926") (unit 1)
+          (reference "C962") (unit 1)
         )
       )
@@
     )
   )
-  (symbol (lib_id "Device:C_Polarized") (at 95.25 120.65 270) (unit 1)
+  (symbol (lib_id "Device:C") (at 95.25 120.65 270) (unit 1)
     (in_bom yes) (on_board yes) (dnp no)
     (property "Reference" "C101" (at 95.25 116.84 90)
@@
       (effects (font (size 1.27 1.27)) (justify left))
     )
-    (property "Value" "0.1uF" (at 128.27 229.87 0)
+    (property "Value" "100nF" (at 128.27 229.87 0)
       (effects (font (size 1.27 1.27)) (justify left))
     )
@@
       (effects (font (size 1.27 1.27)) (justify left))
     )
-    (property "Value" "0.1uF" (at 140.97 229.87 0)
+    (property "Value" "100nF" (at 140.97 229.87 0)
       (effects (font (size 1.27 1.27)) (justify left))
     )
@@
     )
   )
-  (symbol (lib_id "Device:C_Polarized") (at 95.25 97.79 270) (unit 1)
+  (symbol (lib_id "Device:C") (at 95.25 97.79 270) (unit 1)
     (in_bom yes) (on_board yes) (dnp no)
     (property "Reference" "C101" (at 95.25 93.98 90)
